File: cad/fuzz_factory_mod/analog.sch (KiCad schematic (older format))
At the start: 0 parts

Commit message: Added simulation file for DAC + FF.
Continued schematic.
Parts:
- added C?: 10n, symbol Device:C
- added C? (x2): 100n, symbol Device:C
- added C? (x2): 10u, symbol Device:CP
- added Q?: Q_NJFET_DSG, symbol Device:Q_NJFET_DSG
- added Q?: 2N3904, Package_TO_SOT_THT:TO-92_Inline, symbol Transistor_BJT:2N3904
- added Q? (x2): 2N3906, Package_TO_SOT_THT:TO-92_Inline, symbol Transistor_BJT:2N3906
- added R?: 51k, symbol Device:R
- added R? (x3): 4k7, symbol Device:R
- added R?: 1k, symbol Device:R
- added R? (x5): 10k, symbol Device:R
- added R? (x3): 220k, symbol Device:R
- added R?: 5k1, symbol Device:R
- added R?: 470, symbol Device:R
- added R?: 0, symbol Device:R
Connections:
- new net: C?.1, Q?.1 (D), R?.1, R?.1
- new net: Q?.2 (S), R?.1, R?.2
- new net: C?.2, Q?.3 (G), R?.1, R?.2
- new net: C?.2, Q?.3 (C), R?.1, R?.2
- new net: C?.1, Q?.2 (B), R?.2
- new net: C?.2, R?.1 (x2)
- new net: C?.1, Q?.2 (B)
- new net: Q?.2 (B), Q?.3 (C), R?.1
- new net: Q?.3 (C), R?.1
- new net COMP_POT_1: C?.1, Q?.1 (E), R?.1, R?.1, R?.1, R?.2
- new net COMP_POT_2: Q?.1 (E), R?.2, R?.2
- new net DAC_CMD: R?.2
- new net GAIN_POT_2: C?.2, R?.1, R?.2
- new net GATE_POT_1: R?.1, R?.2
- new net GNDA: Q?.1 (E), R?.2, R?.2, R?.2
- new net VOLUME_POT_1: R?.1, R?.2
- new net VOLUME_POT_2: C?.1, R?.1, R?.2
Other:
- note added: "COMP"
- note added: "DNP"
- note added: "GAIN"
- note added: "GATE"
- note added: "VOLUME"
