File: cad/fuzz_factory_mod/PSU.sch (KiCad schematic (older format))
At the start: 27 parts, among them Q2201 BCP51, U2201 TL072, U2202 LM2674M-ADJ, U2203 LM78L05_SO8

Commit message: Continued layout.
Parts:
- C2202, C2206, C2211: value 100uF/25V -> 10u; footprint Capacitors_SMD:CP_Elec_6.3x4.5 -> Capacitors_SMD:CP_Elec_5x5.8
- C2214: footprint Capacitors_SMD:CP_Elec_6.3x4.5 -> Capacitors_SMD:CP_Elec_5x5.8
Connections:
- net GND_ANALOG: now also C2211.2; no longer C2206.2
- net GND_PWR: now also C2206.2; no longer C2211.2
- net VCOM: now also C2211.1; no longer C2206.1
- net at C2201.1, C2203.1, C2212.1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: now also C2206.1; no longer C2211.1
Changed lines of the file:
@@
 EESchema Schematic File Version 4
-LIBS:fuzz_factory_mod-cache
 EELAYER 30 0
 EELAYER END
@@
 	1    0    0    -1
 $EndComp
-$Comp
-L Device:CP C2202
-U 1 1 5E30AEA4
-P 2650 4450
-F 0 "C2202" H 2700 4550 50  0000 L CNN
-F 1 "100uF/25V" H 2200 4350 50  0000 L CNN
-F 2 "Capacitors_SMD:CP_Elec_6.3x4.5" H 2688 4300 50  0001 C CNN
-F 3 "~" H 2650 4450 50  0001 C CNN
-	1    2650 4450
-	1    0    0    -1
-$EndComp
-$Comp
-L Device:CP C2206
-U 1 1 5E30B79A
-P 4600 4450
-F 0 "C2206" H 4718 4496 50  0000 L CNN
-F 1 "100uF/25V" H 4718 4405 50  0000 L CNN
-F 2 "Capacitors_SMD:CP_Elec_6.3x4.5" H 4638 4300 50  0001 C CNN
-F 3 "~" H 4600 4450 50  0001 C CNN
-	1    4600 4450
-	1    0    0    -1
-$EndComp
 Connection ~ 7800 1900
 Wire Wire Line
@@
 $EndComp
 $Comp
-L Device:CP C2211
-U 1 1 5F1281A1
-P 2000 6250
-F 0 "C2211" H 2050 6350 50  0000 L CNN
-F 1 "100uF/25V" H 1450 6200 50  0000 L CNN
-F 2 "Capacitors_SMD:CP_Elec_6.3x4.5" H 2038 6100 50  0001 C CNN
-F 3 "~" H 2000 6250 50  0001 C CNN
-	1    2000 6250
-	1    0    0    -1
-$EndComp
-$Comp
 L Device:C C2213
 U 1 1 5F12A37F
@@
 F 0 "C2214" H 4618 6296 50  0000 L CNN
 F 1 "10u" H 4618 6205 50  0000 L CNN
-F 2 "Capacitors_SMD:CP_Elec_6.3x4.5" H 4538 6100 50  0001 C CNN
+F 2 "Capacitors_SMD:CP_Elec_5x5.8" H 4538 6100 50  0001 C CNN
 F 3 "~" H 4500 6250 50  0001 C CNN
 	1    4500 6250
@@
 Text Notes 5400 6350 0    50   ~ 0
 5V for specific 5V logic\nMIDI
+$Comp
+L Device:CP C?
+U 1 1 5F8085AA
+P 2650 4450
+AR Path="/5DE4AD88/5DF28E5E/5F8085AA" Ref="C?"  Part="1"
+AR Path="/5DE4AD88/5ED499CE/5F8085AA" Ref="C?"  Part="1"
+AR Path="/5E2FAB43/5F8085AA" Ref="C2202"  Part="1"
+F 0 "C2202" H 2768 4496 50  0000 L CNN
+F 1 "10u" H 2768 4405 50  0000 L CNN
+F 2 "Capacitors_SMD:CP_Elec_5x5.8" H 2688 4300 50  0001 C CNN
+F 3 "~" H 2650 4450 50  0001 C CNN
+	1    2650 4450
+	-1   0    0    -1
+$EndComp
+$Comp
+L Device:CP C?
+U 1 1 5F823635
+P 2000 6250
+AR Path="/5DE4AD88/5DF28E5E/5F823635" Ref="C?"  Part="1"
+AR Path="/5DE4AD88/5ED499CE/5F823635" Ref="C?"  Part="1"
+AR Path="/5E2FAB43/5F823635" Ref="C2206"  Part="1"
+F 0 "C2206" H 2118 6296 50  0000 L CNN
+F 1 "10u" H 2118 6205 50  0000 L CNN
+F 2 "Capacitors_SMD:CP_Elec_5x5.8" H 2038 6100 50  0001 C CNN
+F 3 "~" H 2000 6250 50  0001 C CNN
+	1    2000 6250
+	1    0    0    -1
+$EndComp
+$Comp
+L Device:CP C?
+U 1 1 5F8237A2
+P 4600 4450
+AR Path="/5DE4AD88/5DF28E5E/5F8237A2" Ref="C?"  Part="1"
+AR Path="/5DE4AD88/5ED499CE/5F8237A2" Ref="C?"  Part="1"
+AR Path="/5E2FAB43/5F8237A2" Ref="C2211"  Part="1"
+F 0 "C2211" H 4718 4496 50  0000 L CNN
+F 1 "10u" H 4718 4405 50  0000 L CNN
+F 2 "Capacitors_SMD:CP_Elec_5x5.8" H 4638 4300 50  0001 C CNN
+F 3 "~" H 4600 4450 50  0001 C CNN
+	1    4600 4450
+	1    0    0    -1
+$EndComp
 $EndSCHEMATC

Commit message: Continued layout.
Connections:
- net DCDC_VSW: now reaches C2207.2, D2201.1 (K), L2202.1, U2202.8 (VSW)
Changed lines of the file:
@@
 	1    0    0    -1
 $EndComp
+Text Label 6000 1900 0    50   ~ 0
+DCDC_VSW
 $EndSCHEMATC
