File: cad/fuzz_factory_mod/mcu.sch (KiCad schematic (older format))
At the start: 4 parts

Commit message: Continued schematic
Parts:
- removed P? (x2): CONN_NUCLEO_L152RE, symbol flax_lib:CONN_NUCLEO_L152RE
- added R?: R, symbol Device:R
Connections:
- net +3V3: now reaches P?.A16 (+3.3V)
- net +3V3: now also P?.A5 (+3.3V)
- net +5V: now reaches P?.A18 (+5V)
- net GNDD: now reaches P?.A19 (GND)
- net GNDD: now also P?.A20 (GND), P?.A22 (GND), P?.A8 (GND), P?.B20 (GND), P?.B9 (GND)
- net at P?.A24 (VIN): now also R?.2
- new net +9V: R?.1
Changed lines of the file:
@@
 $Descr A4 11693 8268
 encoding utf-8
-Sheet 2 5
+Sheet 2 6
 Title ""
 Date ""
@@
 $EndComp
 $Comp
-L flax_lib:CONN_NUCLEO_L152RE P?
-U 3 1 5DE52036
-P 4350 4200
-F 0 "P?" H 4872 3551 50  0000 L CNN
-F 1 "CONN_NUCLEO_L152RE" H 4872 3460 50  0000 L CNN
-F 2 "" H 5250 2350 50  0000 C CNN
-F 3 "" H 5250 2350 50  0000 C CNN
-	3    4350 4200
-	1    0    0    -1
+L power:+3.3V #PWR?
+U 1 1 5E025882
+P 2600 1400
+F 0 "#PWR?" H 2600 1250 50  0001 C CNN
+F 1 "+3.3V" V 2615 1528 50  0000 L CNN
+F 2 "" H 2600 1400 50  0001 C CNN
+F 3 "" H 2600 1400 50  0001 C CNN
+	1    2600 1400
+	0    -1   -1   0
 $EndComp
 $Comp
-L flax_lib:CONN_NUCLEO_L152RE P?
-U 4 1 5DE54E7B
-P 5650 4200
-F 0 "P?" H 6413 4425 50  0000 C CNN
-F 1 "CONN_NUCLEO_L152RE" H 6413 4334 50  0000 C CNN
-F 2 "" H 6550 2350 50  0000 C CNN
-F 3 "" H 6550 2350 50  0000 C CNN
-	4    5650 4200
-	1    0    0    -1
+L power:+5V #PWR?
+U 1 1 5E026E5A
+P 3850 2000
+F 0 "#PWR?" H 3850 1850 50  0001 C CNN
+F 1 "+5V" V 3865 2128 50  0000 L CNN
+F 2 "" H 3850 2000 50  0001 C CNN
+F 3 "" H 3850 2000 50  0001 C CNN
+	1    3850 2000
+	0    1    1    0
 $EndComp
+Wire Wire Line
+	2700 1400 2600 1400
+$Comp
+L power:GNDD #PWR?
+U 1 1 5E028671
+P 2600 2100
+F 0 "#PWR?" H 2600 1850 50  0001 C CNN
+F 1 "GNDD" V 2604 1990 50  0000 R CNN
+F 2 "" H 2600 2100 50  0001 C CNN
+F 3 "" H 2600 2100 50  0001 C CNN
+	1    2600 2100
+	0    1    1    0
+$EndComp
+$Comp
+L power:GNDD #PWR?
+U 1 1 5E029961
+P 3850 2100
+F 0 "#PWR?" H 3850 1850 50  0001 C CNN
+F 1 "GNDD" V 3854 1990 50  0000 R CNN
+F 2 "" H 3850 2100 50  0001 C CNN
+F 3 "" H 3850 2100 50  0001 C CNN
+	1    3850 2100
+	0    -1   -1   0
+$EndComp
+$Comp
+L power:+9V #PWR?
+U 1 1 5E029C4D
+P 4250 2300
+F 0 "#PWR?" H 4250 2150 50  0001 C CNN
+F 1 "+9V" V 4265 2428 50  0000 L CNN
+F 2 "" H 4250 2300 50  0001 C CNN
+F 3 "" H 4250 2300 50  0001 C CNN
+	1    4250 2300
+	0    1    1    0
+$EndComp
+$Comp
+L Device:R R?
+U 1 1 5E02AB58
+P 4000 2300
+F 0 "R?" V 3793 2300 50  0000 C CNN
+F 1 "R" V 3884 2300 50  0000 C CNN
+F 2 "" V 3930 2300 50  0001 C CNN
+F 3 "~" H 4000 2300 50  0001 C CNN
+	1    4000 2300
+	0    1    -1   0
+$EndComp
+Wire Wire Line
+	4250 2300 4150 2300
+Wire Wire Line
+	2600 2100 2700 2100
+$Comp
+L power:+3.3V #PWR?
+U 1 1 5E03A2B9
+P 3850 1900
+F 0 "#PWR?" H 3850 1750 50  0001 C CNN
+F 1 "+3.3V" V 3865 2028 50  0000 L CNN
+F 2 "" H 3850 1900 50  0001 C CNN
+F 3 "" H 3850 1900 50  0001 C CNN
+	1    3850 1900
+	0    1    1    0
+$EndComp
+$Comp
+L power:GNDD #PWR?
+U 1 1 5E03D33A
+P 3850 2200
+F 0 "#PWR?" H 3850 1950 50  0001 C CNN
+F 1 "GNDD" V 3854 2090 50  0000 R CNN
+F 2 "" H 3850 2200 50  0001 C CNN
+F 3 "" H 3850 2200 50  0001 C CNN
+	1    3850 2200
+	0    -1   -1   0
+$EndComp
+$Comp
+L power:GNDD #PWR?
+U 1 1 5E03FA60
+P 3850 1500
+F 0 "#PWR?" H 3850 1250 50  0001 C CNN
+F 1 "GNDD" V 3854 1390 50  0000 R CNN
+F 2 "" H 3850 1500 50  0001 C CNN
+F 3 "" H 3850 1500 50  0001 C CNN
+	1    3850 1500
+	0    -1   -1   0
+$EndComp
+Wire Wire Line
+	3850 2000 3750 2000
+Wire Wire Line
+	3750 2100 3850 2100
+Wire Wire Line
+	3850 2200 3750 2200
+Wire Wire Line
+	3750 2300 3850 2300
+Wire Wire Line
+	3750 1500 3850 1500
+Wire Wire Line
+	3850 1900 3750 1900
+$Comp
+L power:GNDD #PWR?
+U 1 1 5E04230C
+P 7500 1600
+F 0 "#PWR?" H 7500 1350 50  0001 C CNN
+F 1 "GNDD" V 7504 1490 50  0000 R CNN
+F 2 "" H 7500 1600 50  0001 C CNN
+F 3 "" H 7500 1600 50  0001 C CNN
+	1    7500 1600
+	0    1    1    0
+$EndComp
+Wire Wire Line
+	7600 1600 7500 1600
+$Comp
+L power:GNDD #PWR?
+U 1 1 5E043734
+P 8750 2100
+F 0 "#PWR?" H 8750 1850 50  0001 C CNN
+F 1 "GNDD" V 8754 1990 50  0000 R CNN
+F 2 "" H 8750 2100 50  0001 C CNN
+F 3 "" H 8750 2100 50  0001 C CNN
+	1    8750 2100
+	0    -1   -1   0
+$EndComp
+Wire Wire Line
+	8750 2100 8650 2100
 $EndSCHEMATC
