File: cad/fuzz_factory_mod/mcu.sch (KiCad schematic (older format))
At the start: 24 parts, among them J201 Conn_MCU_SWD, U201 STM32F303VCTx, Y201 Resonator_Small

Commit message: Continued layout.
Changed lines of the file:
@@
 F2 "MIDI_IN" I L 10000 4550 50
 F3 "MIDI_OUT" I L 10000 4650 50
-F4 "+5V" I L 10000 4350 50
+F4 "+5V_IN" I L 10000 4350 50
 $EndSheet
 Text Label 9900 4550 2    50   ~ 0

Commit message: Continued layout.
Connections:
- wire segments 171 -> 170
Changed lines of the file:
@@
 Wire Wire Line
 	2500 3450 3750 3450
-Text Label 5450 4050 0    50   ~ 0
-ENC2_IN_CCW
 Text Label 5450 3950 0    50   ~ 0
 SPI3_MOSI
 Wire Wire Line
 	6500 3950 5350 3950
-Wire Wire Line
-	6500 4050 5350 4050
 Text Label 3650 5850 2    50   ~ 0
-ENC2_IN_CW
+ENC2_IN_CCW
 Text Label 3650 5750 2    50   ~ 0
 ENC2_BTN
