File: cad/fuzz_factory_mod/interface.sch (KiCad schematic (older format))
At the start: 26 parts, among them SW1801 SW_PUSH, U1801 TLC6C598-Q1, U1802 TLC6C598-Q1

Commit message: Continued schematic.
Parts:
- SW501: renamed from SW1801; footprint Pin_Headers:Pin_Header_Straight_1x02 -> Pin_Headers:Pin_Header_Straight_1x02_Pitch2.54mm
- renumbered AFF1801 to AFF501, C1801 to C502, C1802 to C503, C1803 to C504, C1804 to C505, R1801 to R510, R1802 to R511, R1803 to R512, R1804 to R513, R1805 to R514, R1806 to R515, R1807 to R516, R1808 to R517, R1809 to R518, R1810 to R519, R1811 to R520, R1812 to R521, R1813 to R522, R1814 to R523, R1815 to R524, R1816 to R525, R1817 to R526, R1818 to R527, U1801 to U501, U1802 to U502

Commit message: Continued schematic.
Parts:
- removed C504, C505: 100n, Capacitors_SMD:C_0603, symbol Device:C
- removed R526: 100, Resistors_SMD:R_0603, symbol Device:R
- removed R527: 10k, Resistors_SMD:R_0603, symbol Device:R
- removed SW501: SW_PUSH, Pin_Headers:Pin_Header_Straight_1x02_Pitch2.54mm, symbol Switch:SW_Push
Connections:
- net labels removed: FSW_bypass
- wire segments 94 -> 82
Changed lines of the file:
@@
 $Descr A4 11693 8268
 encoding utf-8
-Sheet 5 26
+Sheet 5 30
 Title ""
 Date ""
@@
 Text HLabel 1350 4000 0    60   Input ~ 0
 ENC1_ENC2
-Text HLabel 9100 5550 0    60   Input ~ 0
-FSW_bypass
 $Comp
 L flax_lib:TLC6C598-Q1 U501
@@
 	0    -1   -1   0
 $EndComp
-$Comp
-L Switch:SW_Push SW501
-U 1 1 56FBD957
-P 10050 5550
-F 0 "SW501" H 10200 5660 50  0000 C CNN
-F 1 "SW_PUSH" H 10050 5470 50  0000 C CNN
-F 2 "Pin_Headers:Pin_Header_Straight_1x02_Pitch2.54mm" H 10050 5550 50  0001 C CNN
-F 3 "" H 10050 5550 50  0000 C CNN
-	1    10050 5550
-	1    0    0    -1
-$EndComp
-$Comp
-L Device:C C505
-U 1 1 56FBDE06
-P 9650 5800
-F 0 "C505" H 9675 5900 50  0000 L CNN
-F 1 "100n" H 9675 5700 50  0000 L CNN
-F 2 "Capacitors_SMD:C_0603" H 9688 5650 50  0001 C CNN
-F 3 "" H 9650 5800 50  0000 C CNN
-	1    9650 5800
-	1    0    0    -1
-$EndComp
-$Comp
-L Device:R R526
-U 1 1 56FBE09F
-P 9400 5550
-F 0 "R526" V 9480 5550 50  0000 C CNN
-F 1 "100" V 9400 5550 50  0000 C CNN
-F 2 "Resistors_SMD:R_0603" V 9330 5550 50  0001 C CNN
-F 3 "" H 9400 5550 50  0000 C CNN
-	1    9400 5550
-	0    1    1    0
-$EndComp
-$Comp
-L power:GNDD #PWR0229
-U 1 1 56FBE1C8
-P 9650 6050
-F 0 "#PWR0229" H 9650 5800 50  0001 C CNN
-F 1 "GNDD" H 9650 5900 50  0000 C CNN
-F 2 "" H 9650 6050 50  0000 C CNN
-F 3 "" H 9650 6050 50  0000 C CNN
-	1    9650 6050
-	1    0    0    -1
-$EndComp
-$Comp
-L power:GNDD #PWR0230
-U 1 1 56FBE293
-P 10450 6050
-F 0 "#PWR0230" H 10450 5800 50  0001 C CNN
-F 1 "GNDD" H 10450 5900 50  0000 C CNN
-F 2 "" H 10450 6050 50  0000 C CNN
-F 3 "" H 10450 6050 50  0000 C CNN
-	1    10450 6050
-	1    0    0    -1
-$EndComp
-$Comp
-L Device:R R527
-U 1 1 56FBE7EC
-P 9650 5300
-F 0 "R527" V 9730 5300 50  0000 C CNN
-F 1 "10k" V 9650 5300 50  0000 C CNN
-F 2 "Resistors_SMD:R_0603" V 9580 5300 50  0001 C CNN
-F 3 "" H 9650 5300 50  0000 C CNN
-	1    9650 5300
-	1    0    0    -1
-$EndComp
-$Comp
-L power:+3V3 #PWR0231
-U 1 1 56FBEA4D
-P 9650 5050
-F 0 "#PWR0231" H 9650 4900 50  0001 C CNN
-F 1 "+3V3" H 9650 5190 50  0000 C CNN
-F 2 "" H 9650 5050 50  0000 C CNN
-F 3 "" H 9650 5050 50  0000 C CNN
-	1    9650 5050
-	1    0    0    -1
-$EndComp
-$Comp
-L Device:C C504
-U 1 1 56FC131E
-P 9150 5800
-F 0 "C504" H 9175 5900 50  0000 L CNN
-F 1 "100n" H 9175 5700 50  0000 L CNN
-F 2 "Capacitors_SMD:C_0603" H 9188 5650 50  0001 C CNN
-F 3 "" H 9150 5800 50  0000 C CNN
-	1    9150 5800
-	1    0    0    -1
-$EndComp
-$Comp
-L power:GNDD #PWR0232
-U 1 1 56FC1324
-P 9150 6050
-F 0 "#PWR0232" H 9150 5800 50  0001 C CNN
-F 1 "GNDD" H 9150 5900 50  0000 C CNN
-F 2 "" H 9150 6050 50  0000 C CNN
-F 3 "" H 9150 6050 50  0000 C CNN
-	1    9150 6050
-	1    0    0    -1
-$EndComp
 Wire Wire Line
 	2800 2500 2800 2600
@@
 Wire Wire Line
 	8800 1200 9600 1200
-Wire Wire Line
-	10450 5550 10450 6050
-Wire Wire Line
-	9550 5550 9650 5550
-Wire Wire Line
-	9650 5450 9650 5550
-Connection ~ 9650 5550
-Wire Wire Line
-	9650 5950 9650 6050
-Wire Wire Line
-	9100 5550 9150 5550
-Wire Wire Line
-	9650 5050 9650 5150
-Wire Wire Line
-	9150 5950 9150 6050
-Wire Wire Line
-	9150 5650 9150 5550
-Connection ~ 9150 5550
 $Comp
 L Device:C C503
@@
 $EndComp
 Wire Wire Line
-	9650 5550 9650 5650
-Wire Wire Line
-	9150 5550 9250 5550
-Wire Wire Line
 	8100 750  8100 800
 Wire Wire Line
 	2800 750  2800 800
 Wire Wire Line
-	9650 5550 9850 5550
-Wire Wire Line
-	10250 5550 10450 5550
-Wire Wire Line
 	4200 1200 3500 1200

Commit message: Commit pre- board separation.
Connections:
- net labels added: +3.3V
Changed lines of the file:
@@
-$EndComp
-$Comp
-L power:+3V3 #PWR0227
-U 1 1 56FB7191
-P 2650 3700
-F 0 "#PWR0227" H 2650 3550 50  0001 C CNN
-F 1 "+3V3" H 2650 3840 50  0000 C CNN
-F 2 "" H 2650 3700 50  0000 C CNN
-F 3 "" H 2650 3700 50  0000 C CNN
-	1    2650 3700
-	0    1    1    0
 $EndComp
 $Comp
@@
 $EndComp
 $Comp
-L power:+3V3 #PWR0236
-U 1 1 5E2DCD61
-P 2650 4650
-F 0 "#PWR0236" H 2650 4500 50  0001 C CNN
-F 1 "+3V3" H 2650 4790 50  0000 C CNN
-F 2 "" H 2650 4650 50  0000 C CNN
-F 3 "" H 2650 4650 50  0000 C CNN
-	1    2650 4650
-	0    1    1    0
-$EndComp
-$Comp
 L power:GNDD #PWR0237
 U 1 1 5E2DCD6B
@@
 Wire Wire Line
 	2650 5900 2500 5900
+$Comp
+L power:+3.3V #PWR0262
+U 1 1 5EDC0F01
+P 2650 3700
+F 0 "#PWR0262" H 2650 3550 50  0001 C CNN
+F 1 "+3.3V" V 2665 3828 50  0000 L CNN
+F 2 "" H 2650 3700 50  0001 C CNN
+F 3 "" H 2650 3700 50  0001 C CNN
+	1    2650 3700
+	0    1    1    0
+$EndComp
+$Comp
+L power:+3.3V #PWR0263
+U 1 1 5EDC1B71
+P 2650 4650
+F 0 "#PWR0263" H 2650 4500 50  0001 C CNN
+F 1 "+3.3V" V 2665 4778 50  0000 L CNN
+F 2 "" H 2650 4650 50  0001 C CNN
+F 3 "" H 2650 4650 50  0001 C CNN
+	1    2650 4650
+	0    1    1    0
+$EndComp
 $EndSCHEMATC
