File: cad/fuzz_factory_mod/USB_DEV.sch (KiCad schematic (older format))
At the start: 6 parts, among them J401 USB_B_Micro, U401 USBLC6-2SC6

Commit message: Continued schematic.
Parts:
- U401: footprint Package_TO_SOT_SMD:SOT-23-6 -> TO_SOT_Packages_SMD:SOT-23-6
Changed lines of the file:
@@
 $Descr A4 11693 8268
 encoding utf-8
-Sheet 4 22
+Sheet 4 26
 Title ""
 Date ""
@@
 F 0 "U401" V 4850 3500 50  0000 C CNN
 F 1 "USBLC6-2SC6" V 5550 3700 50  0000 C CNN
-F 2 "Package_TO_SOT_SMD:SOT-23-6" H 4450 3650 50  0001 C CNN
+F 2 "TO_SOT_Packages_SMD:SOT-23-6" H 4450 3650 50  0001 C CNN
 F 3 "http://www2.st.com/resource/en/datasheet/CD00050750.pdf" H 5400 3600 50  0001 C CNN
 	1    5200 3250

Commit message: Continued layout.
Parts:
- U401: symbol Power_Protection:USBLC6-2SC6 -> fuzz_factory_mod-rescue:USBLC6-2SC6-Power_Protection
Changed lines of the file:
@@
 EESchema Schematic File Version 4
-LIBS:fuzz_factory_mod-cache
 EELAYER 30 0
 EELAYER END
@@
 	3700 2850 3700 2800
 $Comp
-L Power_Protection:USBLC6-2SC6 U?
+L fuzz_factory_mod-rescue:USBLC6-2SC6-Power_Protection U?
 U 1 1 5EB62ACF
 P 5200 3250
