File: cad/fuzz_factory_mod/fuzz_factory_mod.kicad_pcb (KiCad board)
At the start: 2 copper layers, 335 parts, among them J1701 Barrel_Jack_Switch, J1702 Conn_Battery, J1703 CONN_AUDIO_OUT, J1704 CONN_AUDIO_IN, J201 Conn_MCU_SWD, J2301 CONN_MIDI_IN, J2302 CONN_MIDI_THRU, J2303 CONN_MIDI_THRU, J301 USB_B_Micro, J401 USB_B_Micro, K1701 EE2-5NU, Q1601 Q_NJFET_DSG, Q1701 DTC114Y, Q1702 DTA114E, Q1901 DTA123Y, Q1902 DTA123Y, Q2001 DTA123Y, Q2002 DTA123Y, Q2101 DTA123Y, Q2102 DTA123Y, Q601 DTA123Y, Q602 DTA123Y, Q603 DTA123Y, Q604 DTA123Y, Q901 Q_NJFET_DSG, SW1901 PEL12D-4225S-S2024, SW2001 PEL12D-4225S-S2024, SW2101 PEL12D-4225S-S2024, U1001 MC33202, U1101 LM1458, U1102 MC33202, U1201 LM2903, U1301 TL072, U1501 LM1458, U1502 MC33202, U1801 TLC6C598-Q1, U1802 TLC6C598-Q1, U201 STM32F303VCTx, U2201 TL072, U2302 4011, U2303 4011, U601 4050, U602 4504, U603 MC33202, U701 AD5262_ABC, U801 TL072

Commit message: Continued schematic.
Parts:
- removed AFF1801: HDSP-521E, flax_lib:AFF_2x7SEG-PT-DIGIT_10mm
- removed C1801, C1802, C1803, C1804, C1901, C1902, C1903, C1904, C2001, C2002, C2003, C2004, C2101, C2102, C2103, C2104: 100n, Capacitors_SMD:C_0603
- removed Q1901, Q1902, Q2001, Q2002, Q2101, Q2102: DTA123Y, TO_SOT_Packages_SMD:SOT-23
- removed R1801, R1802, R1803, R1804, R1805, R1806, R1807, R1808, R1809, R1810, R1811, R1812, R1813, R1814, R1815, R1816: 470, Resistors_SMD:R_0805
- removed R1817, R1902, R1907, R1908, R2002, R2007, R2008, R2102, R2107, R2108: 100, Resistors_SMD:R_0603
- removed R1818, R1901, R1903, R1904, R1905, R1906, R2001, R2003, R2004, R2005, R2006, R2101, R2103, R2104, R2105, R2106: 10k, Resistors_SMD:R_0603
- removed SW1901, SW2001, SW2101: PEL12D-4225S-S2024, flax_lib:PEL12D
- removed U1801, U1802: TLC6C598-Q1, Housings_SOIC:SOIC-16_3.9x9.9mm_Pitch1.27mm
- added AFF501: HDSP-521E, flax_lib:AFF_2x7SEG-PT-DIGIT_10mm, F.Cu at (-81.1, 81.4)
- added C1303: 100n, Capacitors_SMD:C_0603, F.Cu at (149.7, 62.3)
- added C1607: 100n, Capacitors_SMD:C_0603, F.Cu at (108.1, -17.2)
- added C1608: 100n, Capacitors_SMD:C_0603, F.Cu at (128.1, -35.2)
- added C1609: 100n, Capacitors_SMD:C_0603, F.Cu at (93.8, -15.8)
- added C1610: 100n, Capacitors_SMD:C_0603, F.Cu at (119.2, -26.1)
- added C1611: 10u, Capacitors_SMD:CP_Elec_6.3x4.5, F.Cu at (97.1, -20.9)
- added C1612: 100n, Capacitors_SMD:C_0603, F.Cu at (104.3, -17.2)
- added C1613: 100n, Capacitors_SMD:C_0603, F.Cu at (112.8, -19.1)
- added C1614: 100n, Capacitors_SMD:C_0603, F.Cu at (97.7, -15.8)
- added C1615: 100n, Capacitors_SMD:C_0603, F.Cu at (123.6, -30.7)
- added C1702: 1u, Capacitors_SMD:C_0805, F.Cu at (107.1, -9.80)
- added C1703: 100n, Capacitors_SMD:C_0603, F.Cu at (93.8, 2.87)
- added C1704: 100n, Capacitors_SMD:C_0603, F.Cu at (106.9, -7.21)
- added C1705: 100n, Capacitors_SMD:C_0603, F.Cu at (97.7, 2.87)
- added C1706: 220n, Capacitors_SMD:C_0805, F.Cu at (102.7, -5.25)
- added C1707: 100n, Capacitors_SMD:C_0603, F.Cu at (111.3, -10.0)
- added C1708: 100n, Capacitors_SMD:C_0603, F.Cu at (111.3, -7.68)
- added C1709: 100n, Capacitors_SMD:C_0603, F.Cu at (106.9, -4.86)
- added C1710: 100n, Capacitors_SMD:C_0603, F.Cu at (102.3, 0.22)
- added C1805: 1u, Capacitors_SMD:C_0805, F.Cu at (159.1, -26.2)
- added C1806: 100n, Capacitors_SMD:C_0603, F.Cu at (158.8, -20.8)
- added C1807: 100n, Capacitors_SMD:C_0603, F.Cu at (163.3, -25.9)
- added C1808: 100n, Capacitors_SMD:C_0603, F.Cu at (167.8, -28.7)
- added C1809: 220n, Capacitors_SMD:C_0805, F.Cu at (163.6, -30.8)
- added C1810: 100n, Capacitors_SMD:C_0603, F.Cu at (150.3, -18.1)
- added C1811: 100n, Capacitors_SMD:C_0603, F.Cu at (167.8, -31.0)
- added C1812: 100n, Capacitors_SMD:C_0603, F.Cu at (154.1, -18.1)
- added C1813: 100n, Capacitors_SMD:C_0603, F.Cu at (163.3, -28.2)
- added C1905: 100n, Capacitors_SMD:C_0603, F.Cu at (146.6, -3.48)
- added C1906: 100n, Capacitors_SMD:C_0603, F.Cu at (127.9, -3.58)
- added C1907: 100n, Capacitors_SMD:C_0603, F.Cu at (124.1, -1.23)
- added C1908: 100n, Capacitors_SMD:C_0603, F.Cu at (146.6, -5.83)
- added C1909: 100n, Capacitors_SMD:C_0603, F.Cu at (124.1, -3.58)
- added C501: 100n, Capacitors_SMD:C_0603, F.Cu at (306.8, 38.3)
- added C502: 100n, Capacitors_SMD:C_0603, F.Cu at (-51.5, 75.4)
- added C503: 100n, Capacitors_SMD:C_0603, F.Cu at (-56.2, 85.4)
- added C504: 100n, Capacitors_SMD:C_0603, F.Cu at (-52.0, 82.6)
- added C505: 100n, Capacitors_SMD:C_0603, F.Cu at (-56.2, 87.8)
- added C609: 100n, Capacitors_SMD:C_0603, F.Cu at (34.7, -39.4)
- added C610: 100n, Capacitors_SMD:C_0603, F.Cu at (-69.6, 101.7)
- added C611: 100n, Capacitors_SMD:C_0603, F.Cu at (-74.1, 110.8)
- added C612: 100n, Capacitors_SMD:C_0603, F.Cu at (-69.6, 104.0)
- added C613: 100n, Capacitors_SMD:C_0603, F.Cu at (-65.8, 101.7)
- added C703: 100n, Capacitors_SMD:C_0603, F.Cu at (-20.0, 72.5)
- added C704: 100n, Capacitors_SMD:C_0603, F.Cu at (-24.5, 81.6)
- added C705: 100n, Capacitors_SMD:C_0603, F.Cu at (-16.2, 72.5)
- added C706: 100n, Capacitors_SMD:C_0603, F.Cu at (-20.0, 74.8)
- added C803: 100n, Capacitors_SMD:C_0603, F.Cu at (313.0, 24.8)
- added C804: 100n, Capacitors_SMD:C_0603, F.Cu at (-32.5, 101.7)
- added C805: 100n, Capacitors_SMD:C_0603, F.Cu at (-37.0, 110.8)
- added C806: 100n, Capacitors_SMD:C_0603, F.Cu at (-28.7, 101.7)
- added C807: 100n, Capacitors_SMD:C_0603, F.Cu at (-32.5, 104.0)
- added D1102: BZX84Cxx, Diodes_SMD:D_SOT-23_ANK, F.Cu at (257.7, -18.6)
- added D1502: BZX84Cxx, Diodes_SMD:D_SOT-23_ANK, F.Cu at (257.7, -10.7)
- added D1702: BAV23S, TO_SOT_Packages_SMD:SOT-23, F.Cu at (102.6, -8.93)
- added D1703: BZX84Cxx, Diodes_SMD:D_SOT-23_ANK, F.Cu at (269.5, -18.6)
- added D1801: BAV23S, TO_SOT_Packages_SMD:SOT-23, F.Cu at (159.1, -29.9)
- added D1802: BZX84Cxx, Diodes_SMD:D_SOT-23_ANK, F.Cu at (269.5, -10.7)
- added D2201: BAS3010B, Diodes_SMD:D_SOD-323, F.Cu at (41.2, 261.5)
- added D2301: BAT54A, TO_SOT_Packages_SMD:SOT-23, F.Cu at (58.7, 242.3)
- added Q1301: MMDT3904, TO_SOT_Packages_SMD:SOT-363_SC-70-6, F.Cu at (105.1, 223.3)
- added Q1302: MMDT3904, TO_SOT_Packages_SMD:SOT-363_SC-70-6, F.Cu at (109.4, 223.3)
- added Q1602: DTA123Y, TO_SOT_Packages_SMD:SOT-23, F.Cu at (119.5, -34.1)
- added Q1603: DTA123Y, TO_SOT_Packages_SMD:SOT-23, F.Cu at (113.1, -22.6)
- added Q1604: DTA123Y, TO_SOT_Packages_SMD:SOT-23, F.Cu at (123.9, -34.1)
- added Q1605: DTA123Y, TO_SOT_Packages_SMD:SOT-23, F.Cu at (119.5, -29.6)
- added Q2201: BCP51, TO_SOT_Packages_SMD:SOT-223, F.Cu at (74.9, 214.8)
- added Q605: DTA123Y, TO_SOT_Packages_SMD:SOT-23, F.Cu at (-73.8, 107.3)
- added Q606: DTA123Y, TO_SOT_Packages_SMD:SOT-23, F.Cu at (-73.8, 102.8)
- added Q701: DTA123Y, TO_SOT_Packages_SMD:SOT-23, F.Cu at (-24.2, 78.1)
- added Q702: DTA123Y, TO_SOT_Packages_SMD:SOT-23, F.Cu at (-24.2, 73.6)
- added Q801: MMDT3904, TO_SOT_Packages_SMD:SOT-363_SC-70-6, F.Cu at (92.9, 226.2)
- added Q802: MMDT3904, TO_SOT_Packages_SMD:SOT-363_SC-70-6, F.Cu at (97.1, 226.2)
- added Q803: DTA123Y, TO_SOT_Packages_SMD:SOT-23, F.Cu at (-36.7, 102.8)
- added Q804: DTA123Y, TO_SOT_Packages_SMD:SOT-23, F.Cu at (-36.7, 107.3)
- added Q902: DMMT3904W, TO_SOT_Packages_SMD:SOT-363_SC-70-6, F.Cu at (94.0, 212.6)
- added Q903: DMMT3906W, TO_SOT_Packages_SMD:SOT-363_SC-70-6, F.Cu at (94.0, 216.5)
- added Q904: DMMT3906W, TO_SOT_Packages_SMD:SOT-363_SC-70-6, F.Cu at (98.2, 212.6)
- added R1313: 10k, Resistors_SMD:R_0603, F.Cu at (149.5, 64.7)
- added R1617: 4k7, Resistors_SMD:R_0603, F.Cu at (127.9, -32.8)
- added R1618: 4k7, Resistors_SMD:R_0603, F.Cu at (123.5, -28.3)
- added R1619: 4k7, Resistors_SMD:R_0603, F.Cu at (116.5, -19.1)
- added R1620: 4k7, Resistors_SMD:R_0603, F.Cu at (120.6, -23.7)
- added R1621: 0, Resistors_SMD:R_0603, F.Cu at (127.3, -30.3)
- added R1622: 0, Resistors_SMD:R_0603, F.Cu at (117.1, -23.6)
- added R1623: 0, Resistors_SMD:R_0603, F.Cu at (127.0, -27.8)
- added R1624: 0, Resistors_SMD:R_0603, F.Cu at (120.6, -21.2)
- added R1625: 0, Resistors_SMD:R_0603, F.Cu at (124.2, -25.4)
- added R1626: 0, Resistors_SMD:R_0603, F.Cu at (124.2, -20.4)
- added R1627: 1M, Resistors_SMD:R_0603, F.Cu at (115.4, -16.6)
- added R1628: 1M, Resistors_SMD:R_0603, F.Cu at (122.5, -17.9)
- added R1629: 3k9, Resistors_SMD:R_0603, F.Cu at (111.8, -16.7)
- added R1630: 3k9, Resistors_SMD:R_0603, F.Cu at (127.7, -25.4)
- added R1631: 10k, Resistors_SMD:R_0603, F.Cu at (124.2, -22.9)
- added R1632: 10k, Resistors_SMD:R_0603, F.Cu at (118.9, -16.6)
- added R1703: 1k, Resistors_SMD:R_0603, F.Cu at (102.2, 2.63)
- added R1704: 10k, Resistors_SMD:R_0603, F.Cu at (106.3, -2.45)
- added R1705: 10k, Resistors_SMD:R_0603, F.Cu at (117.0, -5.01)
- added R1706: 100k, Resistors_SMD:R_0603, F.Cu at (110.6, -5.27)
- added R1707: 10k, Resistors_SMD:R_0603, F.Cu at (109.9, -2.45)
- added R1708: 10k, Resistors_SMD:R_0603, F.Cu at (115.0, -7.49)
- added R1709: 100k, Resistors_SMD:R_0603, F.Cu at (105.7, 2.76)
- added R1710: 10k, Resistors_SMD:R_0603, F.Cu at (109.6, 0.03)
- added R1711: 10k, Resistors_SMD:R_0805, F.Cu at (102.5, -2.40)
- added R1712: 10k, Resistors_SMD:R_0603, F.Cu at (113.4, -2.79)
- added R1713: 10k, Resistors_SMD:R_0603, F.Cu at (109.3, 2.76)
- added R1714: 10k, Resistors_SMD:R_0603, F.Cu at (113.1, 0.03)
- added R1715: 10k, Resistors_SMD:R_0603, F.Cu at (115.0, -9.97)
- added R1716: 10k, Resistors_SMD:R_0603, F.Cu at (106.0, 0.28)
- added R1819: 1k, Resistors_SMD:R_0603, F.Cu at (165.7, -18.2)
- added R1820: 10k, Resistors_SMD:R_0603, F.Cu at (169.6, -21.0)
- added R1821: 10k, Resistors_SMD:R_0603, F.Cu at (173.4, -26.0)
- added R1822: 100k, Resistors_SMD:R_0603, F.Cu at (171.5, -31.0)
- added R1823: 10k, Resistors_SMD:R_0603, F.Cu at (158.6, -18.4)
- added R1824: 10k, Resistors_SMD:R_0603, F.Cu at (162.5, -20.7)
- added R1825: 100k, Resistors_SMD:R_0603, F.Cu at (167.0, -26.3)
- added R1826: 10k, Resistors_SMD:R_0603, F.Cu at (166.3, -23.4)
- added R1827: 10k, Resistors_SMD:R_0805, F.Cu at (158.9, -23.4)
- added R1828: 10k, Resistors_SMD:R_0603, F.Cu at (171.5, -28.5)
- added R1829: 10k, Resistors_SMD:R_0603, F.Cu at (162.2, -18.2)
- added R1830: 10k, Resistors_SMD:R_0603, F.Cu at (166.0, -21.0)
- added R1831: 10k, Resistors_SMD:R_0603, F.Cu at (169.9, -23.8)
- added R1832: 10k, Resistors_SMD:R_0603, F.Cu at (162.8, -23.4)
- added R1909: 4k7, Resistors_SMD:R_0603, F.Cu at (131.6, -3.52)
- added R1910: 4k7, Resistors_SMD:R_0603, F.Cu at (150.3, -3.29)
- added R1911: 4k7, Resistors_SMD:R_0603, F.Cu at (153.8, -5.77)
- added R1912: 4k7, Resistors_SMD:R_0603, F.Cu at (131.3, -1.04)
- added R1913: 100k, Resistors_SMD:R_0603, F.Cu at (149.2, -0.81)
- added R1914: 100k, Resistors_SMD:R_0603, F.Cu at (127.8, -1.17)
- added R1915: 1k, Resistors_SMD:R_0603, F.Cu at (153.8, -3.29)
- added R1916: 1k, Resistors_SMD:R_0603, F.Cu at (150.3, -5.77)
- added R507: 100k, Resistors_SMD:R_0603, F.Cu at (313.8, 40.9)
- added R508: 0, Resistors_SMD:R_0603, F.Cu at (310.2, 43.4)
- added R509: 10k, Resistors_SMD:R_0603, F.Cu at (314.1, 38.4)
- added R510: 470, Resistors_SMD:R_0805, F.Cu at (-91.0, 92.9)
- added R511: 470, Resistors_SMD:R_0805, F.Cu at (-70.3, 92.9)
- added R512: 470, Resistors_SMD:R_0805, F.Cu at (-74.4, 95.8)
- added R513: 470, Resistors_SMD:R_0805, F.Cu at (-51.9, 79.9)
- added R514: 470, Resistors_SMD:R_0805, F.Cu at (-78.6, 95.8)
- added R515: 470, Resistors_SMD:R_0805, F.Cu at (-74.4, 92.9)
- added R516: 470, Resistors_SMD:R_0805, F.Cu at (-56.0, 82.8)
- added R517: 470, Resistors_SMD:R_0805, F.Cu at (-78.6, 92.9)
- added R518: 470, Resistors_SMD:R_0805, F.Cu at (-82.7, 95.8)
- added R519: 470, Resistors_SMD:R_0805, F.Cu at (-56.0, 79.9)
- added R520: 470, Resistors_SMD:R_0805, F.Cu at (-70.3, 95.8)
- added R521: 470, Resistors_SMD:R_0805, F.Cu at (-82.7, 92.9)
- added R522: 470, Resistors_SMD:R_0805, F.Cu at (-86.9, 95.8)
- added R523: 470, Resistors_SMD:R_0805, F.Cu at (-51.4, 72.7)
- added R524: 470, Resistors_SMD:R_0805, F.Cu at (-86.9, 92.9)
- added R525: 470, Resistors_SMD:R_0805, F.Cu at (-91.0, 95.8)
- added R526: 100, Resistors_SMD:R_0603, F.Cu at (-52.5, 85.5)
- added R527: 10k, Resistors_SMD:R_0603, F.Cu at (-48.3, 82.6)
- added R613: 0, Resistors_SMD:R_0603, F.Cu at (38.1, -36.9)
- added R614: 0, Resistors_SMD:R_0603, F.Cu at (34.5, -34.5)
- added R615: 0, Resistors_SMD:R_0603, F.Cu at (38.4, -39.3)
- added R616: 0, Resistors_SMD:R_0603, F.Cu at (34.5, -37.0)
- added R617: 10k, Resistors_SMD:R_0603, F.Cu at (-62.4, 104.2)
- added R618: 100, Resistors_SMD:R_0603, F.Cu at (-66.2, 106.6)
- added R619: 10k, Resistors_SMD:R_0603, F.Cu at (-74.2, 115.7)
- added R620: 10k, Resistors_SMD:R_0603, F.Cu at (-62.1, 101.8)
- added R621: 10k, Resistors_SMD:R_0603, F.Cu at (-70.4, 110.9)
- added R622: 10k, Resistors_SMD:R_0603, F.Cu at (-74.2, 113.2)
- added R623: 100, Resistors_SMD:R_0603, F.Cu at (-69.8, 106.5)
- added R624: 100, Resistors_SMD:R_0603, F.Cu at (-65.9, 104.1)
- added R701: 10k, Resistors_SMD:R_0603, F.Cu at (-16.6, 77.4)
- added R702: 100, Resistors_SMD:R_0603, F.Cu at (-12.8, 75.0)
- added R703: 10k, Resistors_SMD:R_0603, F.Cu at (-24.6, 86.5)
- added R704: 10k, Resistors_SMD:R_0603, F.Cu at (-12.5, 72.5)
- added R705: 10k, Resistors_SMD:R_0603, F.Cu at (-20.8, 81.6)
- added R706: 10k, Resistors_SMD:R_0603, F.Cu at (-24.6, 84.0)
- added R707: 100, Resistors_SMD:R_0603, F.Cu at (-20.2, 77.2)
- added R708: 100, Resistors_SMD:R_0603, F.Cu at (-16.3, 74.9)
- added R813: 10k, Resistors_SMD:R_0603, F.Cu at (312.9, 27.2)
- added R814: 10k, Resistors_SMD:R_0603, F.Cu at (-25.3, 104.2)
- added R815: 100, Resistors_SMD:R_0603, F.Cu at (-29.1, 106.6)
- added R816: 10k, Resistors_SMD:R_0603, F.Cu at (-37.1, 115.7)
- added R817: 10k, Resistors_SMD:R_0603, F.Cu at (-25.0, 101.8)
- added R818: 10k, Resistors_SMD:R_0603, F.Cu at (-33.3, 110.9)
- added R819: 10k, Resistors_SMD:R_0603, F.Cu at (-32.7, 106.5)
- added R820: 100, Resistors_SMD:R_0603, F.Cu at (-28.8, 104.1)
- added R821: 100, Resistors_SMD:R_0603, F.Cu at (-37.1, 113.2)
- added RV1301: R_POT_TRIM, Potentiometers:Potentiometer_Trimmer_Bourns_3266X, F.Cu at (58.8, -41.7)
- added RV501: 10k, Potentiometers:Potentiometer_Trimmer_Bourns_3266X, F.Cu at (310.2, 40.9)
- added RV502: 10k, Potentiometers:Potentiometer_Trimmer_Bourns_3266X, F.Cu at (306.7, 43.2)
- added RV503: 10k, Potentiometers:Potentiometer_Trimmer_Bourns_3266X, F.Cu at (310.5, 38.4)
- added RV504: 10k, Potentiometers:Potentiometer_Trimmer_Bourns_3266X, F.Cu at (306.7, 40.7)
- added RV801: R_POT_TRIM, Potentiometers:Potentiometer_Trimmer_Bourns_3266X, F.Cu at (305.7, 25.9)
- added SW501: SW_PUSH, Pin_Headers:Pin_Header_Straight_1x02_Pitch2.54mm, F.Cu at (-55.8, 73.6)
- added SW601: PEL12D-4225S-S2024, flax_lib:PEL12D, F.Cu at (-84.5, 108.9)
- added SW701: PEL12D-4225S-S2024, flax_lib:PEL12D, F.Cu at (-34.9, 79.7)
- added SW801: PEL12D-4225S-S2024, flax_lib:PEL12D, F.Cu at (-47.5, 108.9)
- added U1601: 4050, Housings_SOIC:SOIC-16_3.9x9.9mm_Pitch1.27mm, F.Cu at (113.0, -30.6)
- added U1602: 4049, Housings_SOIC:SOIC-16_3.9x9.9mm_Pitch1.27mm, F.Cu at (104.6, -30.6)
- added U1603: 4504, Housings_SOIC:SOIC-16_3.9x9.9mm_Pitch1.27mm, F.Cu at (96.1, -30.6)
- added U1604: MC33202, Housings_SOIC:SOIC-8_3.9x4.9mm_Pitch1.27mm, F.Cu at (106.6, -21.6)
- added U1701: LM1458, Housings_SOIC:SOIC-8_3.9x4.9mm_Pitch1.27mm, F.Cu at (96.2, -1.53)
- added U1702: MC33202, Housings_SOIC:SOIC-8_3.9x4.9mm_Pitch1.27mm, F.Cu at (96.2, -7.98)
- added U1803: LM1458, Housings_SOIC:SOIC-8_3.9x4.9mm_Pitch1.27mm, F.Cu at (152.6, -22.5)
- added U1804: MC33202, Housings_SOIC:SOIC-8_3.9x4.9mm_Pitch1.27mm, F.Cu at (152.6, -29.0)
- added U1901: LM2903, Housings_SOIC:SOIC-8_3.9x4.9mm_Pitch1.27mm, F.Cu at (126.4, -7.98)
- added U2202: LM2674M-ADJ, Housings_SOIC:SOIC-8_3.9x4.9mm_Pitch1.27mm, F.Cu at (35.3, 262.0)
- added U2301: 4N25, Housings_DIP:DIP-6_W7.62mm, F.Cu at (71.6, 226.4)
- added U301: USBLC6-2SC6, TO_SOT_Packages_SMD:SOT-23-6, F.Cu at (98.5, 238.6)
- added U302: FT230XS, Housings_SSOP:SSOP-16_3.9x4.9mm_Pitch0.635mm, F.Cu at (92.1, 239.7)
- added U401: USBLC6-2SC6, TO_SOT_Packages_SMD:SOT-23-6, F.Cu at (107.6, 238.6)
- added U501: TLC6C598-Q1, Housings_SOIC:SOIC-16_3.9x9.9mm_Pitch1.27mm, F.Cu at (-62.3, 88.6)
- added U502: TLC6C598-Q1, Housings_SOIC:SOIC-16_3.9x9.9mm_Pitch1.27mm, F.Cu at (-62.3, 77.1)
- added U604: 4049, Housings_SOIC:SOIC-16_3.9x9.9mm_Pitch1.27mm, F.Cu at (28.5, -34.8)
- added Y201: Resonator_Small, Pin_Headers:Pin_Header_Straight_1x03_Pitch2.54mm, F.Cu at (95.9, 92.7)
- moved J1704 220.7 mm to (266.0, 142.6), turned to 270 degrees
- moved C2209 164.8 mm to (27.5, 265.5)
- moved C2204 159.5 mm to (40.2, 270.3), turned to 180 degrees
- moved C2205 158.5 mm to (41.0, 265.5), turned to 180 degrees
- moved C2207 156.4 mm to (35.4, 258.0)
- moved C2208 154.0 mm to (30.2, 270.3)
- moved R2206 151.9 mm to (29.5, 262.2)
- moved L2201 151.6 mm to (47.0, 262.2), turned to 180 degrees
- moved R2207 144.2 mm to (30.2, 264.7), turned to 270 degrees
- moved J2303 138.1 mm to (-39.9, -15.4)
- moved R2304 138.1 mm to (-71.6, 9.20)
- moved R2305 138.1 mm to (-71.6, 6.32)
- moved J2301 138.1 mm to (-62.4, -15.4)
- moved J2302 138.1 mm to (-17.3, -15.4)
- moved R2301 138.1 mm to (-71.6, 3.44)
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Connections:
- net /ANALOG/ADC_frontend/AN_MCU_1 renamed /ANALOG/fuzz_factory_main/ADC_frontend_1/AN_MCU_1
- net /ANALOG/ADC_frontend/AN_MCU_2 renamed /ANALOG/fuzz_factory_main/ADC_frontend_1/AN_MCU_2
- net /ANALOG/DAC/IN_PWM_LSB_BUFF renamed /ANALOG/DAC1/IN_PWM_LSB_BUFF
- net /ANALOG/DAC/IN_PWM_MSB_BUFF renamed /ANALOG/DAC1/IN_PWM_MSB_BUFF
- net /ANALOG/DAC_CMD renamed /ANALOG/DAC_CMD_1
- net /ANALOG/GAIN_POT_REF_1 renamed /ANALOG/COMP_POT_REF_1
- net /ANALOG/GAIN_POT_REF_3 renamed /ANALOG/COMP_POT_REF_2
- net /ANALOG/IN_PWM_LSBn renamed /ANALOG/DAC1/IN_PWM_LSBn
- net /ANALOG/IN_PWM_MSBn renamed /ANALOG/DAC1/IN_PWM_MSBn
- net /ANALOG/STARVE_POT_1 renamed /ANALOG/fuzz_factory_main/STARVE_POT_1
- net /ANALOG/STARVE_POT_2 renamed /ANALOG/fuzz_factory_main/STARVE_POT_2
- net /ANALOG/freq_meas/OUT_1 renamed /ANALOG/IN_AUDIO_FREQ
- net /ANALOG/freq_meas/OUT_2 renamed /ANALOG/OUT_AUDIO_VCA_FREQ
- net /ANALOG/fuzz_factory_ref/GATE_POT_1 renamed /ANALOG/GATE_POT_REF_1
- net /ANALOG/fuzz_factory_ref/OUT_AUDIO renamed /ANALOG/OUT_AUDIO_REF
- net /ANALOG/fuzz_factory_ref/VOLUME_POT_1 renamed /ANALOG/VOLUME_POT_REF_1
- net /ANALOG/fuzz_factory_ref/VOLUME_POT_2 renamed /ANALOG/VOLUME_POT_REF_2
- net /ANALOG/peak_detect/PEAK_OUT renamed /ANALOG/IN_AUDIO_PEAK
- net /ANALOG/peak_detect/Vsub renamed /ANALOG/peak_detect_audio_in/Vsub
- net /ANALOG/peak_detect2/PEAK_OUT renamed /ANALOG/IN_AUDIO_VCA_PEAK
- net /ANALOG/peak_detect2/Vsub renamed /ANALOG/peak_detect_in_audio_vca/Vsub
- C1101 pad 2: (no net) -> /ANALOG/IN_AUDIO
- C1203 pad 2: (no net) -> /ANALOG/IN_AUDIO
- C1204 pad 2: (no net) -> /ANALOG/OUT_AUDIO
- C1301 pad 2: /ANALOG/VCA2/VCC -> +9V
- C1302 pad 1: /ANALOG/VCA2/Output -> /ANALOG/OUT_AUDIO
- C1501 pad 2: (no net) -> /ANALOG/IN_AUDIO_VCA
- C1604 pad 1: (no net) -> Net-(C1604-Pad1)
- C2207 pad 1: (no net) -> Net-(C2207-Pad1)
- C306 pad 2: (no net) -> Net-(C306-Pad2)
- C801 pad 2: /ANALOG/VCA/VCC -> +9V
- C802 pad 1: /ANALOG/VCA/Output -> /ANALOG/IN_AUDIO_VCA
- C902 pad 2: /ANALOG/IN_AUDIO -> /ANALOG/IN_AUDIO_VCA
- C903 pad 1: /ANALOG/IN_AUDIO -> /ANALOG/IN_AUDIO_VCA
- C904 pad 1: (no net) -> Net-(C904-Pad1)
- J301 pad 2: (no net) -> Net-(J301-Pad2)
- J301 pad 3: (no net) -> Net-(J301-Pad3)
- J401 pad 1: (no net) -> Net-(J401-Pad1)
- J401 pad 2: (no net) -> Net-(J401-Pad2)
- J401 pad 3: (no net) -> Net-(J401-Pad3)
- Q601 pad 1: /ANALOG/IN_PWM_LSB -> FF_Stab_DAC_PWM_LSB
- Q603 pad 1: /ANALOG/IN_PWM_MSB -> FF_Stab_DAC_PWM_MSB
- R1301 pad 2: (no net) -> /ANALOG/OUT_AUDIO
- R1302 pad 2: /ANALOG/VCA2/VCC -> +9V
- R1304 pad 2: (no net) -> Net-(Q1301-Pad3)
- R1305 pad 1: (no net) -> Net-(R1305-Pad1)
- R1306 pad 2: (no net) -> Net-(R1306-Pad2)
- R1307 pad 2: /ANALOG/VCA2/VCC -> +9V
- R1311 pad 2: /ANALOG/VCA2/VCC -> +9V
- R1312 pad 1: /ANALOG/VCA2/Output -> /ANALOG/OUT_AUDIO
- R1601 pad 2: (no net) -> /ANALOG/DAC_CMD_2
- R1608 pad 1: (no net) -> Net-(Q903-Pad3)
- R1612 pad 1: (no net) -> Net-(Q904-Pad3)
- R202 pad 1: (no net) -> Net-(R202-Pad1)
- R2201 pad 1: (no net) -> +BATT
- R2301 pad 1: (no net) -> Net-(D2301-Pad2)
- R301 pad 1: (no net) -> Net-(R301-Pad1)
- R302 pad 1: (no net) -> Net-(R302-Pad1)
- R303 pad 2: (no net) -> Net-(R303-Pad2)
- R304 pad 2: (no net) -> Net-(R304-Pad2)
- R607 pad 2: /ANALOG/DAC/IN_PWM_LSBn_BUFF -> /ANALOG/DAC1/IN_PWM_LSBn_BUFF
- R609 pad 2: /ANALOG/DAC/IN_PWM_MSBn_BUFF -> /ANALOG/DAC1/IN_PWM_MSBn_BUFF
- R801 pad 2: (no net) -> /ANALOG/IN_AUDIO
- R802 pad 2: /ANALOG/VCA/VCC -> +9V
- R804 pad 2: (no net) -> Net-(Q801-Pad3)
- R805 pad 1: (no net) -> Net-(R805-Pad1)
- R806 pad 2: (no net) -> Net-(R806-Pad2)
- R807 pad 2: /ANALOG/VCA/VCC -> +9V
- R811 pad 2: /ANALOG/VCA/VCC -> +9V
- R812 pad 1: /ANALOG/VCA/Output -> /ANALOG/IN_AUDIO_VCA
- R908 pad 1: (no net) -> Net-(Q903-Pad6)
- R912 pad 1: (no net) -> Net-(Q904-Pad6)
- U1301 pad 1: /ANALOG/VCA2/Output -> /ANALOG/OUT_AUDIO
- U1301 pad 5: (no net) -> /ANALOG/VCA2/CV
- U1301 pad 8: /ANALOG/VCA2/VCC -> +9V
- U201 pad 1: (no net) -> VCA_IN_PWM
- U201 pad 2: (no net) -> VCA_OUT_PWM
- U201 pad 3: (no net) -> /MCU/ENC1_LED_RED
- U201 pad 30: (no net) -> SPI_FF_Gain_SCK
- U201 pad 31: (no net) -> SPI_FF_Gain_MISO
- U201 pad 35: (no net) -> SPI_FF_Gain_CS
- U201 pad 4: (no net) -> /MCU/ENC1_LED_GREEN
- U201 pad 40: (no net) -> FF_Stab_DAC_PWM_LSB
- U201 pad 42: (no net) -> FF_Stab_DAC_PWM_MSB
- U201 pad 44: (no net) -> Ref_Stab_DAC_PWM_LSB
- U201 pad 45: (no net) -> Ref_Stab_DAC_PWM_MSB
- U201 pad 52: (no net) -> /MCU/SPI2_SCK
- U201 pad 54: (no net) -> /MCU/SPI2_MOSI
- U201 pad 7: (no net) -> /MCU/ENC1_BTN
- U201 pad 8: (no net) -> /MCU/ENC1_IN_CW
- U201 pad 84: (no net) -> /MCU/ENC2_LED_RED
- U201 pad 85: (no net) -> /MCU/ENC2_LED_GREEN
- U201 pad 87: (no net) -> /MCU/ENC2_BTN
- U201 pad 88: (no net) -> /MCU/ENC2_IN_CW
- U201 pad 9: (no net) -> /MCU/ENC1_IN_CCW
- U201 pad 92: (no net) -> /MCU/ENC2_IN_CCW
- U601 pad 10: /ANALOG/DAC/IN_PWM_MSBn_BUFF -> /ANALOG/DAC1/IN_PWM_MSBn_BUFF
- U601 pad 4: /ANALOG/DAC/IN_PWM_LSBn_BUFF -> /ANALOG/DAC1/IN_PWM_LSBn_BUFF
- U602 pad 10: /ANALOG/DAC/IN_PWM_MSBn_BUFF -> Net-(R615-Pad2)
- U602 pad 3: /ANALOG/IN_PWM_LSB -> FF_Stab_DAC_PWM_LSB
- U602 pad 4: /ANALOG/DAC/IN_PWM_LSBn_BUFF -> Net-(R613-Pad2)
- U602 pad 7: /ANALOG/IN_PWM_MSB -> FF_Stab_DAC_PWM_MSB
- U701 pad 10: (no net) -> /ANALOG/Digipot/~DIGIPOT_PR
- U701 pad 6: (no net) -> /ANALOG/Digipot/~DIGIPOT_SHDN
- U701 pad 7: (no net) -> SPI_FF_Gain_SCK
- U701 pad 8: (no net) -> SPI_FF_Gain_MISO
- U701 pad 9: (no net) -> SPI_FF_Gain_CS
- U801 pad 1: /ANALOG/VCA/Output -> /ANALOG/IN_AUDIO_VCA
- U801 pad 5: (no net) -> /ANALOG/VCA/CV
- U801 pad 8: /ANALOG/VCA/VCC -> +9V

Commit message: Continued schematic.
Parts:
- removed C504, C505: 100n, Capacitors_SMD:C_0603
- removed D2301: BAT54A, TO_SOT_Packages_SMD:SOT-23
- removed J2301: CONN_MIDI_IN, flax_lib:DIN5_through_hole
- removed J2302, J2303: CONN_MIDI_THRU, flax_lib:DIN5_through_hole
- removed R2301, R2304, R2305, R2306, R2307: 220, Resistors_SMD:R_0805
- removed R2302: 4k7, Resistors_SMD:R_0603
- removed R2303, R526: 100, Resistors_SMD:R_0603
- removed R527: 10k, Resistors_SMD:R_0603
- removed SW501: SW_PUSH, Pin_Headers:Pin_Header_Straight_1x02_Pitch2.54mm
- removed U2301: 4N25, Housings_DIP:DIP-6_W7.62mm
- removed U2302, U2303: 4011, Housings_SOIC:SOIC-14_3.9x8.7mm_Pitch1.27mm
- added C1110: 100n, Capacitors_SMD:C_0603, F.Cu at (-241.4, 21.4)
- added C1111: 100n, Capacitors_SMD:C_0603, F.Cu at (-241.4, 23.8)
- added C1206: 100n, Capacitors_SMD:C_0603, F.Cu at (-241.4, 32.0)
- added C1207: 100n, Capacitors_SMD:C_0603, F.Cu at (-241.4, 34.3)
- added C1304: 100n, Capacitors_SMD:C_0603, F.Cu at (-225.0, 23.8)
- added C1305: 100n, Capacitors_SMD:C_0603, F.Cu at (-225.0, 21.4)
- added C907: 100n, Capacitors_SMD:C_0603, F.Cu at (-114.2, -10.0)
- added D901: BAT54A, TO_SOT_Packages_SMD:SOT-23, F.Cu at (-134.8, -11.2)
- added J901: CONN_MIDI_IN, flax_lib:DIN5_through_hole, F.Cu at (-129.8, -26.8)
- added J902: CONN_MIDI_THRU, flax_lib:DIN5_through_hole, F.Cu at (-105.5, -26.2)
- added J903: CONN_MIDI_OUT, flax_lib:DIN5_through_hole, F.Cu at (-82.7, -26.2)
- added R1115: 100, Resistors_SMD:R_0603, F.Cu at (-237.7, 21.5)
- added R1116: 10k, Resistors_SMD:R_0603, F.Cu at (-241.6, 26.2)
- added R1209: 100, Resistors_SMD:R_0603, F.Cu at (-241.6, 36.7)
- added R1210: 10k, Resistors_SMD:R_0603, F.Cu at (-237.7, 32.0)
- added R1314: 100, Resistors_SMD:R_0603, F.Cu at (-225.2, 26.2)
- added R1315: 10k, Resistors_SMD:R_0603, F.Cu at (-221.3, 21.5)
- added R917: 220, Resistors_SMD:R_0805, F.Cu at (-125.8, -18.2)
- added R918: 4k7, Resistors_SMD:R_0603, F.Cu at (-119.2, -11.5)
- added R919: 100, Resistors_SMD:R_0603, F.Cu at (-102.2, -12.0)
- added R920: 220, Resistors_SMD:R_0805, F.Cu at (-99.5, -16.8)
- added R921: 220, Resistors_SMD:R_0805, F.Cu at (-109.5, -16.8)
- added R922: 220, Resistors_SMD:R_0805, F.Cu at (-76.8, -17.0)
- added R923: 220, Resistors_SMD:R_0805, F.Cu at (-86.8, -16.8)
- added SW1101: SW_PUSH, Pin_Headers:Pin_Header_Straight_1x02_Pitch2.54mm, F.Cu at (-245.7, 22.6)
- added SW1201: SW_PUSH, Pin_Headers:Pin_Header_Straight_1x02_Pitch2.54mm, F.Cu at (-245.7, 33.1)
- added SW1301: SW_PUSH, Pin_Headers:Pin_Header_Straight_1x02_Pitch2.54mm, F.Cu at (-229.3, 22.6)
- added U901: 4N25, Housings_DIP:DIP-6_W7.62mm, F.Cu at (-130.2, -12.8)
- added U902: 4011, Housings_SOIC:SOIC-14_3.9x8.7mm_Pitch1.27mm, F.Cu at (-108.5, -9.95)
- moved J1701 314.0 mm to (14.8, 284.8)
- moved C1701 278.6 mm to (-3.47, 272.3)
- moved J1702 278.6 mm to (9.78, 259.5)
- moved K1701 278.6 mm to (-1.99, 262.8)
- moved Q701 119.1 mm to (-119.9, 148.9)
- moved R701 119.1 mm to (-112.4, 148.1)
- moved R702 119.1 mm to (-108.5, 145.8)
- moved R703 119.1 mm to (-120.4, 157.2)
- moved R705 119.1 mm to (-116.5, 152.4)
- moved R706 119.1 mm to (-120.4, 154.7)
- moved R707 119.1 mm to (-115.9, 148.0)
- moved R708 119.1 mm to (-112.1, 145.6)
- moved C703 119.1 mm to (-115.8, 143.2)
- moved C704 119.1 mm to (-120.2, 152.3)
- moved C705 119.1 mm to (-111.9, 143.2)
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Connections:
- AFF501 pad 13: (no net) -> +5V
- AFF501 pad 5: +5V -> Net-(AFF501-Pad5)
- Q1701 pad 1: (no net) -> BYPASS_CMD
- R522 pad 2: (no net) -> Net-(AFF501-Pad5)
- U201 pad 10: (no net) -> /MCU/SW_BYPASS
- U201 pad 11: (no net) -> BYPASS_CMD
- U201 pad 80: (no net) -> /MCU/UART5_TX
- U201 pad 83: (no net) -> /MCU/UART5_RX
- U201 pad 97: (no net) -> /MCU/SW_PRESET_UP
- U201 pad 98: (no net) -> /MCU/SW_PRESET_DOWN

Commit message: Continued schematic.
Continued component placement.
Parts:
- added C1901: 100p, Capacitors_SMD:C_0603, F.Cu at (45.0, 80.0)
- added C210: 100n, Capacitors_SMD:C_0603, F.Cu at (92.4, 40.7)
- added C211: 100n, Capacitors_SMD:C_0603, F.Cu at (92.4, 43.0)
- added C212: 100n, Capacitors_SMD:C_0603, F.Cu at (96.3, 40.7)
- added C2210: 100p, Capacitors_SMD:C_0603, F.Cu at (42.5, 179.5)
- added C2401: 100n, Capacitors_SMD:C_0603, F.Cu at (79.2, 139.4)
- added C2402: 100n, Capacitors_SMD:C_0603, F.Cu at (87.7, 132.9)
- added C2403: 100n, Capacitors_SMD:C_0603, F.Cu at (83.0, 139.4)
- added C2501: 100p, Capacitors_SMD:C_0603, F.Cu at (265.5, 118.5)
- added C2601: 100p, Capacitors_SMD:C_0603, F.Cu at (77.8, 215.9)
- added J2801: CONN_AUDIO_OUT_REF, Connect:NMJ6HCD2, F.Cu at (310.8, 152.8)
- added J2802: CONN_EXP_1, Connect:NMJ6HCD2, F.Cu at (-15.5, 119.0)
- added J2803: CONN_EXP_2, Connect:NMJ6HCD2, F.Cu at (-15.5, 98.2)
- added R204: 0, Resistors_SMD:R_0603, F.Cu at (96.1, 43.1)
- added R2401: 1k, Resistors_SMD:R_0603, F.Cu at (87.5, 135.3)
- added R2402: 1k, Resistors_SMD:R_0603, F.Cu at (91.4, 133.0)
- added R2403: 10k, Resistors_SMD:R_0603, F.Cu at (86.7, 139.4)
- added R2404: 10k, Resistors_SMD:R_0603, F.Cu at (91.1, 135.5)
- added R2405: 10k, Resistors_SMD:R_0603, F.Cu at (90.3, 138.0)
- added R2406: 10k, Resistors_SMD:R_0603, F.Cu at (90.3, 140.4)
- added R2801: 1k, Resistors_SMD:R_0603, F.Cu at (9.25, 110.2)
- added R2802: 1k, Resistors_SMD:R_0603, F.Cu at (8.50, 106.9)
- added R2803: 1k, Resistors_SMD:R_0603, F.Cu at (8.75, 103.2)
- added R2804: 1k, Resistors_SMD:R_0603, F.Cu at (8.00, 90.0)
- added R2805: 1k, Resistors_SMD:R_0603, F.Cu at (8.00, 92.5)
- added R2806: 1k, Resistors_SMD:R_0603, F.Cu at (8.25, 95.5)
- added U2401: MC33202, Housings_SOIC:SOIC-8_3.9x4.9mm_Pitch1.27mm, F.Cu at (81.5, 135.0)
- AFF501, SW601, SW701, SW801: moved to B.Cu
- J1703: value CONN_AUDIO_OUT -> CONN_AUDIO_IN
- J1704: value CONN_AUDIO_IN -> CONN_AUDIO_OUT
- Y201: footprint Pin_Headers:Pin_Header_Straight_1x03_Pitch2.54mm -> flax_lib:Resonator_AEL_ZTTxx_SMD
- moved J901 450.6 mm to (305.8, 88.8), turned to 270 degrees
- moved C1110 437.6 mm to (143.6, 229.5), turned to 180 degrees
- moved R917 437.3 mm to (297.2, 92.8), turned to 270 degrees
- moved C1304 436.1 mm to (159.5, 229.5), turned to 180 degrees
- moved D901 435.5 mm to (290.2, 83.8), turned to 180 degrees
- moved C1305 435.3 mm to (158.8, 227.0), turned to 270 degrees
- moved SW1101 435.2 mm to (139.3, 225.6)
- moved SW1301 435.2 mm to (155.7, 225.6)
- moved R1116 435.2 mm to (144.5, 227.0), turned to 90 degrees
- moved C1111 434.4 mm to (142.5, 227.0), turned to 270 degrees
- moved U901 433.9 mm to (291.8, 88.2), turned to 270 degrees
- moved R1315 433.8 mm to (160.8, 227.0), turned to 90 degrees
- moved J902 433.7 mm to (305.2, 113.0), turned to 270 degrees
- moved R1314 432.8 mm to (159.5, 224.5)
- moved R1115 431.7 mm to (143.2, 224.5)
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Connections:
- net /ANALOG/DAC1/IN_PWM_LSB_BUFF renamed /ANALOG/DAC/IN_PWM_LSB_BUFF
- net /ANALOG/DAC1/IN_PWM_LSBn renamed /ANALOG/DAC/IN_PWM_LSBn
- net /ANALOG/DAC1/IN_PWM_LSBn_BUFF renamed /ANALOG/DAC/IN_PWM_LSBn_BUFF
- net /ANALOG/DAC1/IN_PWM_MSB_BUFF renamed /ANALOG/DAC/IN_PWM_MSB_BUFF
- net /ANALOG/DAC1/IN_PWM_MSBn renamed /ANALOG/DAC/IN_PWM_MSBn
- net /ANALOG/DAC1/IN_PWM_MSBn_BUFF renamed /ANALOG/DAC/IN_PWM_MSBn_BUFF
- net /ANALOG/DAC2/IN_PWM_LSB_BUFF renamed /ANALOG/DAC_REF/IN_PWM_LSB_BUFF
- net /ANALOG/DAC2/IN_PWM_LSBn renamed /ANALOG/DAC_REF/IN_PWM_LSBn
- net /ANALOG/DAC2/IN_PWM_LSBn_BUFF renamed /ANALOG/DAC_REF/IN_PWM_LSBn_BUFF
- net /ANALOG/DAC2/IN_PWM_MSB_BUFF renamed /ANALOG/DAC_REF/IN_PWM_MSB_BUFF
- net /ANALOG/DAC2/IN_PWM_MSBn renamed /ANALOG/DAC_REF/IN_PWM_MSBn
- net /ANALOG/DAC2/IN_PWM_MSBn_BUFF renamed /ANALOG/DAC_REF/IN_PWM_MSBn_BUFF
- net /ANALOG/DAC_CMD_1 renamed /ANALOG/DAC_CMD
- net /ANALOG/DAC_CMD_2 renamed /ANALOG/DAC_CMD_REF
- net /ANALOG/OUT_AUDIO_REF renamed AUDIO_REF_OUT_FX
- net /ANALOG/VCA/CV renamed /ANALOG/VCA_IN/CV
- net /ANALOG/VCA2/CV renamed /ANALOG/VCA_OUT/CV
- net Net-(C1604-Pad1) renamed /ANALOG/fuzz_factory_ref/POL_MEAS_2
- net Net-(C1604-Pad2) renamed /ANALOG/fuzz_factory_ref/POL_MEAS_1
- C1002 pad 1: /ANALOG/fuzz_factory_main/ADC_frontend_1/AN_MCU_1 -> ADC_FF_pol1
- C1003 pad 1: /ANALOG/fuzz_factory_main/ADC_frontend_1/AN_MCU_2 -> ADC_FF_pol2
- C1101 pad 2: /ANALOG/IN_AUDIO -> AUDIO_IN_FX
- C1203 pad 2: /ANALOG/IN_AUDIO -> AUDIO_IN_FX
- C1204 pad 2: /ANALOG/OUT_AUDIO -> AUDIO_OUT_FX
- C1302 pad 1: /ANALOG/OUT_AUDIO -> AUDIO_OUT_FX
- C1701 pad 1: /CONNECTORS/BATT -> +BATT
- C1702 pad 2: /ANALOG/OUT_AUDIO -> AUDIO_OUT_FX
- C1805 pad 2: /ANALOG/OUT_AUDIO -> AUDIO_OUT_FX
- C904 pad 1: Net-(C904-Pad1) -> /ANALOG/fuzz_factory_main/POL_MEAS_2
- C904 pad 2: Net-(C904-Pad2) -> /ANALOG/fuzz_factory_main/POL_MEAS_1
- C906 pad 2: /ANALOG/OUT_AUDIO -> AUDIO_OUT_FX
- J1701 pad 2: /CONNECTORS/BATT -> +BATT
- K1701 pad 5: (no net) -> AUDIO_OUT_FX
- K1701 pad 8: (no net) -> AUDIO_IN_FX
- NT1701 pad 2: GNDS -> GNDA
- Q1702 pad 2: /CONNECTORS/BATT -> +BATT
- Q902 pad 6: Net-(C904-Pad2) -> /ANALOG/fuzz_factory_main/POL_MEAS_1
- Q903 pad 2: Net-(C904-Pad1) -> /ANALOG/fuzz_factory_main/POL_MEAS_2
- R1001 pad 2: (no net) -> /ANALOG/fuzz_factory_main/POL_MEAS_1
- R1002 pad 2: (no net) -> /ANALOG/fuzz_factory_main/POL_MEAS_2
- R1003 pad 2: /ANALOG/fuzz_factory_main/ADC_frontend_1/AN_MCU_1 -> ADC_FF_pol1
- R1004 pad 1: /ANALOG/fuzz_factory_main/ADC_frontend_1/AN_MCU_1 -> ADC_FF_pol1
- R1005 pad 2: /ANALOG/fuzz_factory_main/ADC_frontend_1/AN_MCU_2 -> ADC_FF_pol2
- R1006 pad 1: /ANALOG/fuzz_factory_main/ADC_frontend_1/AN_MCU_2 -> ADC_FF_pol2
- R1207 pad 2: /ANALOG/IN_AUDIO_FREQ -> INPUT_CAPTURE_1
- R1208 pad 2: /ANALOG/OUT_AUDIO_VCA_FREQ -> INPUT_CAPTURE_2
- R1301 pad 2: /ANALOG/OUT_AUDIO -> AUDIO_OUT_FX
- R1312 pad 1: /ANALOG/OUT_AUDIO -> AUDIO_OUT_FX
- R1916 pad 2: /ANALOG/OUT_AUDIO_REF_FREQ -> INPUT_CAPTURE_3
- R801 pad 2: /ANALOG/IN_AUDIO -> AUDIO_IN_FX
- R905 pad 2: Net-(C904-Pad2) -> /ANALOG/fuzz_factory_main/POL_MEAS_1
- R906 pad 1: Net-(C904-Pad2) -> /ANALOG/fuzz_factory_main/POL_MEAS_1
- R916 pad 1: /ANALOG/OUT_AUDIO -> AUDIO_OUT_FX
- U1201 pad 1: /ANALOG/IN_AUDIO_FREQ -> INPUT_CAPTURE_1
- U1201 pad 7: /ANALOG/OUT_AUDIO_VCA_FREQ -> INPUT_CAPTURE_2
- U1301 pad 1: /ANALOG/OUT_AUDIO -> AUDIO_OUT_FX
- U1901 pad 7: /ANALOG/OUT_AUDIO_REF_FREQ -> INPUT_CAPTURE_3
- U201 pad 14: (no net) -> /MCU/NRST
- U201 pad 24: (no net) -> ADC_FF_pol1
- U201 pad 25: (no net) -> ADC_FF_pol2
- U201 pad 27: (no net) -> EXP_1
- U201 pad 33: (no net) -> EXP_2
- U201 pad 48: (no net) -> /MCU/DISP_ENABLE
- U201 pad 59: (no net) -> INPUT_CAPTURE_1
- U201 pad 93: (no net) -> /MCU/DISP_LATCH
- U201 pad 95: (no net) -> INPUT_CAPTURE_2
- U201 pad 96: (no net) -> INPUT_CAPTURE_3
- U501 pad 12: /MCU/interface/DISP_LATCH -> /MCU/DISP_LATCH
- U501 pad 13: /MCU/interface/DISP_ENABLE -> /MCU/DISP_ENABLE
- U502 pad 12: /MCU/interface/DISP_LATCH -> /MCU/DISP_LATCH
- U502 pad 13: /MCU/interface/DISP_ENABLE -> /MCU/DISP_ENABLE

Commit message: Commit pre- board separation.
Parts:
- added J1301: Conn_analog_1, Pin_Headers:Pin_Header_Straight_1x06_Pitch2.54mm, F.Cu at (159.2, 90.8)
- added J1302: Conn_analog_2, Pin_Headers:Pin_Header_Straight_1x06_Pitch2.54mm, F.Cu at (182.8, 90.5)
- added J202: Conn_interface_1, Pin_Headers:Pin_Header_Straight_1x12_Pitch2.54mm_SMD_Pin1Left, F.Cu at (64.8, 39.0)
- added J203: Conn_interface_2, Pin_Headers:Pin_Header_Straight_1x12_Pitch2.54mm_SMD_Pin1Left, F.Cu at (207.5, 48.0)
- moved C2601 228.1 mm to (266.8, 88.0)
Connections:
- C610 pad 2: /MCU/ENC1_BTN -> /MCU/interface/ENC1_SW
- C612 pad 2: /MCU/ENC1_IN_CCW -> /MCU/interface/ENC1_ENC2
- C613 pad 2: /MCU/ENC1_IN_CW -> /MCU/interface/ENC1_ENC1
- C703 pad 2: /MCU/ENC2_BTN -> /MCU/interface/ENC2_SW
- C705 pad 2: /MCU/ENC2_IN_CCW -> /MCU/interface/ENC2_ENC2
- C706 pad 2: /MCU/ENC2_IN_CW -> /MCU/interface/ENC2_ENC1
- Q605 pad 1: /MCU/ENC1_LED_GREEN -> (no net)
- Q606 pad 1: /MCU/ENC1_LED_RED -> (no net)
- Q701 pad 1: /MCU/ENC2_LED_GREEN -> (no net)
- Q702 pad 1: /MCU/ENC2_LED_RED -> (no net)
- R618 pad 2: /MCU/ENC1_BTN -> /MCU/interface/ENC1_SW
- R623 pad 1: /MCU/ENC1_IN_CCW -> /MCU/interface/ENC1_ENC2
- R624 pad 1: /MCU/ENC1_IN_CW -> /MCU/interface/ENC1_ENC1
- R702 pad 2: /MCU/ENC2_BTN -> /MCU/interface/ENC2_SW
- R707 pad 1: /MCU/ENC2_IN_CCW -> /MCU/interface/ENC2_ENC2
- R708 pad 1: /MCU/ENC2_IN_CW -> /MCU/interface/ENC2_ENC1
- U501 pad 11: /MCU/SPI2_SCK -> /MCU/interface/DISP_CLK
- U501 pad 12: /MCU/DISP_LATCH -> /MCU/interface/DISP_LATCH
- U501 pad 13: /MCU/DISP_ENABLE -> /MCU/interface/DISP_ENABLE
- U501 pad 14: /MCU/SPI2_MOSI -> (no net)
- U502 pad 11: /MCU/SPI2_SCK -> /MCU/interface/DISP_CLK
- U502 pad 12: /MCU/DISP_LATCH -> /MCU/interface/DISP_LATCH
- U502 pad 13: /MCU/DISP_ENABLE -> /MCU/interface/DISP_ENABLE
