File: cad/fuzz_factory_mod/fuzz_factory_mod.kicad_pcb (KiCad board)
At the start: 2 copper layers, 516 parts, among them J1301 Conn_analog_1, J1302 Conn_analog_2, J1701 Barrel_Jack_Switch, J1702 Conn_Battery, J1703 CONN_AUDIO_IN, J1704 CONN_AUDIO_OUT, J201 Conn_MCU_SWD, J202 Conn_interface_1, J203 Conn_interface_2, J2801 CONN_AUDIO_OUT_REF, J2802 CONN_EXP_1, J2803 CONN_EXP_2, J301 USB_B_Micro, J401 USB_B_Micro, J901 CONN_MIDI_IN, J902 CONN_MIDI_THRU, J903 CONN_MIDI_OUT, K1701 EE2-5NU, Q1301 MMDT3904, Q1302 MMDT3904, Q1601 Q_NJFET_DSG, Q1602 DTA123Y, Q1603 DTA123Y, Q1604 DTA123Y, Q1605 DTA123Y, Q1701 DTC114Y, Q1702 DTA114E, Q2201 BCP51, Q601 DTA123Y, Q602 DTA123Y, Q603 DTA123Y, Q604 DTA123Y, Q605 DTA123Y, Q606 DTA123Y, Q701 DTA123Y, Q702 DTA123Y, Q801 MMDT3904, Q802 MMDT3904, Q803 DTA123Y, Q804 DTA123Y, Q901 Q_NJFET_DSG, Q902 DMMT3904W, Q903 DMMT3906W, Q904 DMMT3906W, SW1101 SW_PUSH, SW1201 SW_PUSH, SW1301 SW_PUSH, SW601 PEL12D-4225S-S2024, SW701 PEL12D-4225S-S2024, SW801 PEL12D-4225S-S2024, U1001 MC33202, U1101 LM1458, U1102 MC33202, U1201 LM2903, U1301 TL072, U1501 LM1458, U1502 MC33202, U1601 4050, U1602 4049, U1603 4504, U1604 MC33202, U1701 LM1458, U1702 MC33202, U1803 LM1458, U1804 MC33202, U1901 LM2903, U201 STM32F303VCTx, U2201 TL072, U2202 LM2674M-ADJ, U2401 MC33202, U301 USBLC6-2SC6, U302 FT230XS, U401 USBLC6-2SC6, U501 TLC6C598-Q1, U502 TLC6C598-Q1, U601 4050, U602 4504, U603 MC33202, U604 4049, U701 AD5262_ABC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

Commit message: Changes architecture.
Corrections on schematic.
Continued Layout placement.
Parts:
- removed AFF501: HDSP-521E, flax_lib:AFF_2x7SEG-PT-DIGIT_10mm
- removed C1001, C1002, C1003, C1603, C1604, C2401, C2402, C2403, C502, C503, C610, C611, C612, C613, C703, C704, C705, C706, C804, C805, C806, C807, C903, C904: 100n, Capacitors_SMD:C_0603
- removed C1601, C901: 10n, Capacitors_SMD:C_0603
- removed C1602, C1605, C1606, C902, C905, C906: 10u, Capacitors_SMD:CP_Elec_6.3x4.5
- removed J1301: Conn_analog_1, Pin_Headers:Pin_Header_Straight_1x06_Pitch2.54mm
- removed J1302: Conn_analog_2, Pin_Headers:Pin_Header_Straight_1x06_Pitch2.54mm
- removed J202: Conn_interface_1, Pin_Headers:Pin_Header_Straight_1x12_Pitch2.54mm_SMD_Pin1Left
- removed J203: Conn_interface_2, Pin_Headers:Pin_Header_Straight_1x12_Pitch2.54mm_SMD_Pin1Left
- removed K1701: EE2-5NU, flax_lib:RELAY-EE2
- removed NT1701: Net-Tie_2, Oddities:NetTie-II
- removed Q1601, Q901: Q_NJFET_DSG, TO_SOT_Packages_SMD:SOT-23
- removed Q605, Q606, Q701, Q702, Q803, Q804: DTA123Y, TO_SOT_Packages_SMD:SOT-23
- removed Q902: DMMT3904W, TO_SOT_Packages_SMD:SOT-363_SC-70-6
- removed Q903, Q904: DMMT3906W, TO_SOT_Packages_SMD:SOT-363_SC-70-6
- removed R1001, R1002, R1601, R2401, R2402, R901: 1k, Resistors_SMD:R_0603
- removed R1003, R1004, R1005, R1006, R1605, R1609, R1610, R1611, R1615, R2403, R2404, R2405, R2406, R617, R619, R620, R621, R622, R701, R703, R704, R705, R706, R816, R817, R818, R819, R905, R909, R910, R911, R915: 10k, Resistors_SMD:R_0603
- removed R1602, R902: 51k, Resistors_SMD:R_0603
- removed R1603, R1604, R903, R904: 0, Resistors_SMD:R_0603
- removed R1606, R1616, R906, R916: 220k, Resistors_SMD:R_0603
- removed R1607, R1613, R1614, R907, R913, R914: 4k7, Resistors_SMD:R_0603
- removed R1608, R908: 470, Resistors_SMD:R_0603
- removed R1612, R912: 5k1, Resistors_SMD:R_0603
- removed R507: 100k, Resistors_SMD:R_0603
- removed R510, R511, R512, R513, R514, R515, R516, R517, R518, R519, R520, R521, R522, R523, R524, R525: 470, Resistors_SMD:R_0805
- removed R618, R623, R624, R702, R707, R708, R820, R821: 100, Resistors_SMD:R_0603
- removed RV501, RV502, RV503, RV504: 10k, Potentiometers:Potentiometer_Trimmer_Bourns_3266X
- removed SW601, SW701, SW801: PEL12D-4225S-S2024, flax_lib:PEL12D
- removed U1001, U2401: MC33202, Housings_SOIC:SOIC-8_3.9x4.9mm_Pitch1.27mm
- removed U1301, U801: TL072, Housings_SOIC:SOIC-8_3.9x4.9mm_Pitch1.27mm
- removed U502: TLC6C598-Q1, Housings_SOIC:SOIC-16_3.9x9.9mm_Pitch1.27mm
- removed U902: 4011, Housings_SOIC:SOIC-14_3.9x8.7mm_Pitch1.27mm
- added C1112: 1u, Capacitors_SMD:C_0805, B.Cu at (11.2, 238.8)
- added C1208: 1u, Capacitors_SMD:C_0805, F.Cu at (-208.5, 104.0)
- added C1510: 1u, Capacitors_SMD:C_0805, F.Cu at (-28.8, 105.8)
- added C2211: 100uF/25V, Capacitors_SMD:CP_Elec_6.3x4.5, F.Cu at (40.8, -29.0)
- added C2212: 100nF, Capacitors_SMD:C_0603, F.Cu at (40.5, -23.8)
- added C2213: 100nF, Capacitors_SMD:C_0603, F.Cu at (30.5, -23.2)
- added C2214: 10u, Capacitors_SMD:CP_Elec_6.3x4.5, F.Cu at (30.8, -29.0)
- added J101: Conn_interface_1, Pin_Headers:Pin_Header_Straight_1x16_Pitch2.54mm_SMD_Pin1Left, F.Cu at (-140.2, 99.2)
- added J102: Conn_interface_2, Pin_Headers:Pin_Header_Straight_1x16_Pitch2.54mm_SMD_Pin1Left, F.Cu at (-92.2, 98.8)
- added J904: Conn_01x10_Female, Pin_Headers:Pin_Header_Straight_1x10_Pitch2.54mm, F.Cu at (-91.2, 194.6)
- added J905: Conn_01x10_Female, Pin_Headers:Pin_Header_Straight_1x10_Pitch2.54mm, F.Cu at (-86.5, 194.6)
- added K2101: Fujitsu-Takamisawa-A_AL, Relays_ThroughHole:Relay_DPDT_FRT5, F.Cu at (-182.5, 74.8)
- added R1316: 10k, Resistors_SMD:R_0603, F.Cu at (-26.5, 100.2)
- added R1317: 10k, Resistors_SMD:R_0603, F.Cu at (-17.0, 100.2)
- added R205: 0, Resistors_SMD:R_0603, F.Cu at (-165.2, 101.2)
- added R206: 0, Resistors_SMD:R_0603, F.Cu at (-163.2, 101.2)
- added R207: 100, Resistors_SMD:R_0603, F.Cu at (-122.2, 110.2)
- added R208: 100, Resistors_SMD:R_0603, F.Cu at (-117.8, 110.2)
- added R2101: 200, Resistors_SMD:R_0805, F.Cu at (-168.2, 74.5)
- added U1202: MC33202, Housings_SOIC:SOIC-8_3.9x4.9mm_Pitch1.27mm, F.Cu at (-215.0, 86.0)
- added U1503: MC33202, Housings_SOIC:SOIC-8_3.9x4.9mm_Pitch1.27mm, F.Cu at (-11.2, 99.1)
- added U2203: LM78L05_SO8, Housings_SOIC:SOIC-8_3.9x4.9mm_Pitch1.27mm, F.Cu at (35.5, -22.5)
- C1701: value 47u -> 100uF/25V
- C201, C202, C203, C204, C205, C206, C207, C208, C209, C305, C306, C701, L201, Q1602, Q1603, Q1604, Q1605, R1617, R1618, R1619, R1620, R303, R304, U302: moved to B.Cu
- C303: footprint Capacitors_SMD:CP_Elec_6.3x4.5 -> Capacitors_SMD:C_1206; moved to B.Cu
- J1703, J1704, J2801, J2802, J2803: footprint Connect:NMJ6HCD2 -> flax_lib:CLIFF_FCR5005x
- R2206: value 10k -> 82k
- R2207: value 10k -> 47k
- R815: value 100 -> 10k
- U501: value TLC6C598-Q1 -> 74LS132; footprint Housings_SOIC:SOIC-16_3.9x9.9mm_Pitch1.27mm -> Housings_SOIC:SOIC-14_3.9x8.7mm_Pitch1.27mm
- moved D1701 508.7 mm to (-181.5, 63.5), turned to 270 degrees
- moved Q1701 504.1 mm to (-177.5, 63.5), turned to 270 degrees
- moved R1702 491.1 mm to (-174.0, 64.2), turned to 180 degrees
- moved R1701 482.8 mm to (-165.8, 78.5)
- moved J901 481.6 mm to (-173.8, 133.2), turned to 90 degrees
- moved J903 481.3 mm to (-173.8, 88.0), turned to 90 degrees
- moved J2801 480.3 mm to (-158.5, 50.2), turned to 180 degrees
- moved J902 479.0 mm to (-173.8, 110.8), turned to 90 degrees
- moved R922 465.6 mm to (-165.8, 82.0), turned to 270 degrees
- moved J1704 464.5 mm to (-136.8, 50.2), turned to 180 degrees
- moved R917 464.1 mm to (-165.8, 124.0), turned to 90 degrees
- moved R923 461.5 mm to (-164.5, 97.5), turned to 0 degrees
- moved R920 461.2 mm to (-165.2, 104.8), turned to 270 degrees
- moved R921 461.0 mm to (-165.2, 114.8), turned to 90 degrees
- moved U901 459.2 mm to (-165.0, 135.5), turned to 90 degrees
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Connections:
- C1908 pad 2: AUDIO_REF_OUT_FX -> /ANALOG/OUT_AUDIO_REF
- C210 pad 1: EXP_1 -> Net-(C210-Pad1)
- C211 pad 1: EXP_2 -> Net-(C211-Pad1)
- D1701 pad 1: Net-(D1701-Pad1) -> (no net)
- D1701 pad 2: (no net) -> Net-(D1701-Pad2)
- J2801 pad 3: AUDIO_REF_OUT_FX -> (no net)
- Q1301 pad 4: GNDA -> Net-(Q1301-Pad1)
- Q1301 pad 5: Net-(Q1301-Pad3) -> Net-(Q1301-Pad5)
- Q1302 pad 2: Net-(Q1301-Pad3) -> Net-(Q1302-Pad2)
- Q1302 pad 3: Net-(Q1302-Pad3) -> Net-(Q1302-Pad2)
- Q1302 pad 4: Net-(Q1301-Pad1) -> GNDA
- Q1302 pad 5: Net-(Q1302-Pad5) -> Net-(Q1302-Pad2)
- Q1701 pad 3: Net-(D1701-Pad1) -> Net-(D1701-Pad3)
- Q1702 pad 1: Net-(NT1701-Pad1) -> GNDA
- Q801 pad 4: GNDA -> Net-(Q801-Pad1)
- Q801 pad 5: Net-(Q801-Pad3) -> Net-(Q801-Pad5)
- Q802 pad 2: Net-(Q801-Pad3) -> Net-(Q802-Pad2)
- Q802 pad 3: Net-(Q802-Pad3) -> Net-(Q802-Pad2)
- Q802 pad 4: Net-(Q801-Pad1) -> GNDA
- Q802 pad 5: Net-(Q802-Pad5) -> Net-(Q802-Pad2)
- R1301 pad 2: AUDIO_OUT_FX -> Net-(C1510-Pad1)
- R1304 pad 2: Net-(Q1301-Pad3) -> Net-(Q1302-Pad2)
- R1306 pad 1: Net-(Q1302-Pad3) -> Net-(Q1301-Pad3)
- R1307 pad 1: Net-(Q1302-Pad5) -> Net-(Q1301-Pad5)
- R1308 pad 1: Net-(Q1302-Pad5) -> Net-(Q1301-Pad5)
- R1310 pad 1: Net-(Q1302-Pad3) -> Net-(Q1301-Pad3)
- R501 pad 1: /ANALOG/COMP_POT_1 -> /ANALOG/GAIN_POT_1
- R502 pad 1: /ANALOG/COMP_POT_2 -> /ANALOG/GAIN_POT_3
- R503 pad 1: /ANALOG/COMP_POT_REF_1 -> /ANALOG/GAIN_POT_REF_1
- R504 pad 1: /ANALOG/COMP_POT_REF_2 -> /ANALOG/GAIN_POT_REF_3
- R801 pad 2: AUDIO_IN_FX -> Net-(C1208-Pad1)
- R804 pad 2: Net-(Q801-Pad3) -> Net-(Q802-Pad2)
- R806 pad 1: Net-(Q802-Pad3) -> Net-(Q801-Pad3)
- R807 pad 1: Net-(Q802-Pad5) -> Net-(Q801-Pad5)
- R808 pad 1: Net-(Q802-Pad5) -> Net-(Q801-Pad5)
- R810 pad 1: Net-(Q802-Pad3) -> Net-(Q801-Pad3)
- R814 pad 1: +5V -> Net-(Q801-Pad2)
- R814 pad 2: Net-(Q803-Pad3) -> +9V
- R815 pad 1: Net-(C805-Pad2) -> Net-(Q801-Pad5)
- R815 pad 2: /MCU/interface/ENC3_SW -> +9V
- R918 pad 2: +3V3 -> +5V
- U201 pad 3: /MCU/ENC1_LED_RED -> ENC1__LED_RED
- U201 pad 4: /MCU/ENC1_LED_GREEN -> ENC1__LED_GREEN
- U201 pad 48: /MCU/DISP_ENABLE -> DISP_ENABLE
- U201 pad 52: /MCU/SPI2_SCK -> SPI2_SCK
- U201 pad 54: /MCU/SPI2_MOSI -> SPI2_MOSI
- U201 pad 55: (no net) -> ENC3_BTN
- U201 pad 56: (no net) -> ENC3_LED_RED
- U201 pad 57: (no net) -> ENC3_LED_GREEN
- U201 pad 58: (no net) -> ENC3_IN_CW
- U201 pad 60: (no net) -> ENC3_IN_CCW
- U201 pad 7: /MCU/ENC1_BTN -> ENC1_BTN
- U201 pad 8: /MCU/ENC1_IN_CW -> ENC1_IN_CW
- U201 pad 82: (no net) -> ENC2_IN_CCW
- U201 pad 84: /MCU/ENC2_LED_RED -> ENC2_LED_RED
- U201 pad 85: /MCU/ENC2_LED_GREEN -> ENC2_LED_GREEN
- U201 pad 87: /MCU/ENC2_BTN -> ENC2_BTN
- U201 pad 88: /MCU/ENC2_IN_CW -> ENC2_IN_CCW
- U201 pad 9: /MCU/ENC1_IN_CCW -> ENC1_IN_CCW
- U201 pad 92: /MCU/ENC2_IN_CCW -> ENC2_IN_CCW
- U201 pad 93: /MCU/DISP_LATCH -> DISP_LATCH
- U501 pad 1: Net-(R511-Pad2) -> /MCU/UART5_RX
- U501 pad 10: +5V -> /MCU/UART5_TX
- U501 pad 11: /MCU/interface/DISP_CLK -> Net-(R923-Pad2)
- U501 pad 12: /MCU/interface/DISP_LATCH -> Net-(U501-Pad12)
- U501 pad 13: /MCU/interface/DISP_ENABLE -> Net-(U501-Pad12)
- U501 pad 14: (no net) -> +5V
- U501 pad 2: Net-(R512-Pad2) -> /MCU/UART5_RX
- U501 pad 3: Net-(R513-Pad2) -> Net-(U501-Pad3)
- U501 pad 4: Net-(R514-Pad2) -> Net-(U501-Pad3)
- U501 pad 5: Net-(R515-Pad2) -> Net-(U501-Pad3)
- U501 pad 6: Net-(R516-Pad2) -> Net-(R921-Pad2)
- U501 pad 7: Net-(R517-Pad2) -> GNDD
- U501 pad 8: GNDD -> Net-(U501-Pad12)
- U501 pad 9: /MCU/interface/shift1_data_out_int -> /MCU/UART5_TX
- U901 pad 6: +3V3 -> +5V
Other:
- board outline added: 138 x 114 mm

Commit message: Continued layout placement.
Parts:
- moved C2201 209.4 mm to (-78.2, 95.5), turned to 180 degrees
- moved C2202 204.0 mm to (-78.2, 88.2), turned to 180 degrees
- moved C401 200.8 mm to (-57.8, 143.0), turned to 90 degrees
- moved R401 198.6 mm to (-60.2, 140.2), turned to 0 degrees
- moved R402 196.0 mm to (-60.2, 138.2), turned to 0 degrees
- moved U401 195.2 mm to (-56.5, 139.2), turned to 180 degrees
- moved J401 192.0 mm to (-51.0, 138.9), turned to 90 degrees
- moved C2208 191.2 mm to (-52.2, 116.2), turned to 90 degrees
- moved C402 191.0 mm to (-57.8, 135.5), turned to 270 degrees
- moved R2202 190.1 mm to (-50.2, 91.0), turned to 0 degrees
- moved Q2201 187.4 mm to (-57.0, 88.2)
- moved R2201 187.3 mm to (-50.2, 89.2), turned to 180 degrees
- moved R2203 185.4 mm to (-62.5, 92.2)
- moved C2203 185.2 mm to (-63.2, 94.5)
- moved C2209 185.1 mm to (-53.2, 107.8), turned to 90 degrees
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Routing:
- net /ANALOG/IN_AUDIO_VCA: track 0.00 -> 4.12 mm
- net Net-(C802-Pad2): track 0.00 -> 4.08 mm
- net +9V: track 0.00 -> 1.97 mm
Other:
- net class Default: clearance 0.2 -> 0.15; trace_width 0.25 -> 0.15; via_dia 0.8 -> 0.6; via_drill 0.4 -> 0.35
- rule trace_clearance: 0.2 -> 0.15
- rule trace_min: 0.2 -> 0.15
- rule via_min_drill: 0.3 -> 0.35
- rule via_min_size: 0.4 -> 0.6

Commit message: Updated trimmers footprint.
Continued layout.
Parts:
- removed C1611, C605: 10u, Capacitors_SMD:CP_Elec_6.3x4.5
- Q601, Q602, Q603, Q604, R601, R602, R603, R604: moved to B.Cu
- RV1301, RV801: footprint Potentiometers:Potentiometer_Trimmer_Bourns_3266X -> Potentiometers:Potentiometer_Trimmer_Piher_PT-10v10_Horizontal_Px10.0mm_Py5.0mm
- moved C501 235.4 mm to (-102.8, 119.2)
- moved R508 231.3 mm to (-113.0, 116.0), turned to 180 degrees
- moved R509 228.9 mm to (-100.2, 118.5), turned to 90 degrees
- moved C1112 172.1 mm to (-107.2, 114.0)
- moved C701 172.1 mm to (-107.2, 115.8)
- moved C702 172.1 mm to (-102.0, 115.2)
- moved R501 172.1 mm to (-112.0, 110.0)
- moved R502 172.1 mm to (-108.5, 110.0)
- moved R503 172.1 mm to (-106.8, 110.0)
- moved R504 172.1 mm to (-103.2, 110.0)
- moved R505 172.1 mm to (-105.0, 110.0)
- moved R506 172.1 mm to (-110.2, 110.0)
- moved U701 172.1 mm to (-107.2, 115.0)
- moved J904 84.2 mm to (-136.2, 123.5)
- moved J905 71.5 mm to (-94.0, 123.5)
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
Commit message: Continued layout.
Parts:
- removed R1109, R1509, R1711, R1827: 10k, Resistors_SMD:R_0805
- added R1318: 10k, Resistors_SMD:R_0603, F.Cu at (-153.5, 118.0)
- added R1601: 10k, Resistors_SMD:R_0603, F.Cu at (-155.5, 148.8)
- added R1801: 10k, Resistors_SMD:R_0603, F.Cu at (-144.0, 124.2)
- added R1901: 10k, Resistors_SMD:R_0603, F.Cu at (-98.0, 155.0)
- C201, C202, C203, C204, C205, C206, C207, C208, C209, L201, R1617: moved to F.Cu
- C2202, C2206, C2211: value 100uF/25V -> 10u; footprint Capacitors_SMD:CP_Elec_6.3x4.5 -> Capacitors_SMD:CP_Elec_5x5.8
- C2214: footprint Capacitors_SMD:CP_Elec_6.3x4.5 -> Capacitors_SMD:CP_Elec_5x5.8
- RV1301, RV801: moved to B.Cu
- moved R612 259.1 mm to (-130.4, 141.7), turned to 0 degrees
- moved R611 256.1 mm to (-127.7, 141.7), turned to 0 degrees
- moved U603 252.2 mm to (-128.8, 136.3), turned to 270 degrees
- moved C608 249.6 mm to (-125.0, 138.1), turned to 270 degrees
- moved C606 241.8 mm to (-122.8, 140.2), turned to 90 degrees
- moved R605 240.7 mm to (-105.3, 120.4), turned to 90 degrees
- moved C601 240.6 mm to (-109.3, 123.9), turned to 90 degrees
- moved C604 240.5 mm to (-122.8, 137.0), turned to 90 degrees
- moved R606 239.2 mm to (-103.6, 120.4), turned to 90 degrees
- moved R609 238.0 mm to (-122.8, 134.0), turned to 90 degrees
- moved C602 236.6 mm to (-109.3, 127.7), turned to 270 degrees
- moved U602 232.7 mm to (-102.9, 125.8), turned to 90 degrees
- moved R610 230.2 mm to (-112.5, 134.4)
- moved C603 230.1 mm to (-112.4, 136.1)
- moved R608 229.4 mm to (-112.5, 139.4)
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Connections:
- C2206 pad 1: VCOM -> Net-(C2201-Pad1)
- C2206 pad 2: GNDA -> GNDD
- C2211 pad 1: Net-(C2201-Pad1) -> VCOM
- C2211 pad 2: GNDD -> GNDA
- R303 pad 1: (no net) -> /MCU/USART1_TX
- R304 pad 1: (no net) -> /MCU/USART1_RX
- U201 pad 34: (no net) -> /MCU/USART1_RX
- U201 pad 68: (no net) -> /MCU/USART1_TX
Routing:
- net +3V3: track 0.00 -> 88.2 mm, vias 0 -> 2
- net /ANALOG/DAC_REF/IN_PWM_MSB_BUFF: track 0.00 -> 29.6 mm, vias 0 -> 2
- net Net-(R1623-Pad2): track 0.00 -> 29.2 mm, vias 0 -> 2
- net +3.3VA: track 0.00 -> 28.0 mm
- net /ANALOG/DAC_REF/IN_PWM_LSBn_BUFF: track 0.00 -> 25.3 mm, vias 0 -> 2
- net Net-(Q1602-Pad3): track 0.00 -> 25.2 mm, vias 0 -> 3
- net /ANALOG/DAC_REF/IN_PWM_MSBn_BUFF: track 0.00 -> 25.1 mm, vias 0 -> 2
- net Net-(C1706-Pad2): track 0.00 -> 22.7 mm
- net Net-(C1809-Pad2): track 0.00 -> 22.6 mm
- net /MCU/NRST: track 0.00 -> 21.9 mm, vias 0 -> 2
- net +9V: track 1.97 -> 22.9 mm, vias 0 -> 2
- net Net-(C1705-Pad1): track 0.00 -> 20.0 mm, vias 0 -> 2
- net Net-(C1808-Pad1): track 0.00 -> 19.5 mm, vias 0 -> 2
- net /ANALOG/DAC_REF/IN_PWM_LSB_BUFF: track 0.00 -> 18.3 mm, vias 0 -> 1
- net GNDA: track 0.00 -> 17.6 mm, vias 0 -> 4
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- added copper zone on B.Cu, net GNDA
- added copper zone on F.Cu, net GNDA
- added copper zone on F.Cu, net GNDD
