File: cad/fuzz_factory_mod/peak_detect.sch (KiCad schematic (older format))
At the start: 28 parts, among them U1101 LM1458, U1102 MC33202

Commit message: Continued layout.
Changed lines of the file:
@@
 $Descr A4 11693 8268
 encoding utf-8
-Sheet 18 22
+Sheet 13 22
 Title ""
 Date ""
@@
 AR Path="/5DE4AD88/5EE3A0D9/5E68F0EA" Ref="U1701"  Part="1"
 AR Path="/5DE4AD88/5EE3A870/5E68F0EA" Ref="U1803"  Part="1"
-F 0 "U1803" H 4500 1600 50  0000 L CNN
+F 0 "U1101" H 4500 1600 50  0000 L CNN
 F 1 "LM1458" H 4500 1500 50  0000 L CNN
 F 2 "Housings_SOIC:SOIC-8_3.9x4.9mm_Pitch1.27mm" H 4400 1400 50  0001 C CNN
@@
 AR Path="/5DE4AD88/5EE3A0D9/5E6962AD" Ref="C1703"  Part="1"
 AR Path="/5DE4AD88/5EE3A870/5E6962AD" Ref="C1806"  Part="1"
-F 0 "C1806" V 4298 1000 50  0000 C CNN
+F 0 "C1102" V 4298 1000 50  0000 C CNN
 F 1 "100n" V 4389 1000 50  0000 C CNN
 F 2 "Capacitors_SMD:C_0603" H 4588 850 50  0001 C CNN
@@
 AR Path="/5DE4AD88/5EE3A0D9/5E698A36" Ref="D1702"  Part="1"
 AR Path="/5DE4AD88/5EE3A870/5E698A36" Ref="D1801"  Part="1"
-F 0 "D1801" H 5100 1923 50  0000 C CNN
+F 0 "D1101" H 5100 1923 50  0000 C CNN
 F 1 "BAV23S" H 5100 2014 50  0000 C CNN
 F 2 "TO_SOT_Packages_SMD:SOT-23" H 5100 1800 50  0001 C CNN
@@
 AR Path="/5DE4AD88/5EE3A0D9/5E69B280" Ref="R1706"  Part="1"
 AR Path="/5DE4AD88/5EE3A870/5E69B280" Ref="R1822"  Part="1"
-F 0 "R1822" V 5150 2150 50  0000 C CNN
+F 0 "R1104" V 5150 2150 50  0000 C CNN
 F 1 "100k" V 5350 2200 50  0000 C CNN
 F 2 "Resistors_SMD:R_0603" V 5180 2200 50  0001 C CNN
@@
 AR Path="/5DE4AD88/5EE3A0D9/5E69DA20" Ref="R1703"  Part="1"
 AR Path="/5DE4AD88/5EE3A870/5E69DA20" Ref="R1819"  Part="1"
-F 0 "R1819" V 3450 1450 50  0000 C CNN
+F 0 "R1101" V 3450 1450 50  0000 C CNN
 F 1 "1k" V 3650 1500 50  0000 C CNN
 F 2 "Resistors_SMD:R_0603" V 3480 1500 50  0001 C CNN
@@
 AR Path="/5DE4AD88/5EE3A0D9/5E69F7E3" Ref="C1705"  Part="1"
 AR Path="/5DE4AD88/5EE3A870/5E69F7E3" Ref="C1808"  Part="1"
-F 0 "C1808" V 5100 2600 50  0000 C CNN
+F 0 "C1104" V 5100 2600 50  0000 C CNN
 F 1 "100n" V 5400 2600 50  0000 C CNN
 F 2 "Capacitors_SMD:C_0603" H 5288 2450 50  0001 C CNN
@@
 AR Path="/5DE4AD88/5EE3A0D9/5E6A149A" Ref="R1704"  Part="1"
 AR Path="/5DE4AD88/5EE3A870/5E6A149A" Ref="R1820"  Part="1"
-F 0 "R1820" V 3900 2500 50  0000 C CNN
+F 0 "R1102" V 3900 2500 50  0000 C CNN
 F 1 "10k" V 4100 2450 50  0000 C CNN
 F 2 "Resistors_SMD:R_0603" V 3930 2450 50  0001 C CNN
@@
 AR Path="/5DE4AD88/5EE3A0D9/5E6A62ED" Ref="C1706"  Part="1"
 AR Path="/5DE4AD88/5EE3A870/5E6A62ED" Ref="C1809"  Part="1"
-F 0 "C1809" H 6115 2296 50  0000 L CNN
+F 0 "C1105" H 6115 2296 50  0000 L CNN
 F 1 "220n" H 6115 2205 50  0000 L CNN
 F 2 "Capacitors_SMD:C_0805" H 6038 2100 50  0001 C CNN
@@
 AR Path="/5DE4AD88/5EE3A0D9/5E6A8BC8" Ref="R1708"  Part="1"
 AR Path="/5DE4AD88/5EE3A870/5E6A8BC8" Ref="R1824"  Part="1"
-F 0 "R1824" V 6150 1750 50  0000 C CNN
+F 0 "R1106" V 6150 1750 50  0000 C CNN
 F 1 "10k" V 6350 1800 50  0000 C CNN
 F 2 "Resistors_SMD:R_0603" V 6180 1800 50  0001 C CNN
@@
 AR Path="/5DE4AD88/5EE3A0D9/5E6A985A" Ref="C1707"  Part="1"
 AR Path="/5DE4AD88/5EE3A870/5E6A985A" Ref="C1810"  Part="1"
-F 0 "C1810" H 6615 2296 50  0000 L CNN
+F 0 "C1106" H 6615 2296 50  0000 L CNN
 F 1 "100n" H 6615 2205 50  0000 L CNN
 F 2 "Capacitors_SMD:C_0603" H 6538 2100 50  0001 C CNN
@@
 AR Path="/5DE4AD88/5EE3A0D9/5E6AA988" Ref="R1709"  Part="1"
 AR Path="/5DE4AD88/5EE3A870/5E6AA988" Ref="R1825"  Part="1"
-F 0 "R1825" V 6900 2000 50  0000 C CNN
+F 0 "R1107" V 6900 2000 50  0000 C CNN
 F 1 "100k" V 7100 2050 50  0000 C CNN
 F 2 "Resistors_SMD:R_0603" V 6930 2050 50  0001 C CNN
@@
 AR Path="/5DE4AD88/5EE3A0D9/5E6AE15B" Ref="R1707"  Part="1"
 AR Path="/5DE4AD88/5EE3A870/5E6AE15B" Ref="R1823"  Part="1"
-F 0 "R1823" V 5650 2000 50  0000 C CNN
+F 0 "R1105" V 5650 2000 50  0000 C CNN
 F 1 "10k" V 5850 2050 50  0000 C CNN
 F 2 "Resistors_SMD:R_0603" V 5680 2050 50  0001 C CNN
@@
 AR Path="/5DE4AD88/5EE3A0D9/5E6B33E4" Ref="U1702"  Part="1"
 AR Path="/5DE4AD88/5EE3A870/5E6B33E4" Ref="U1804"  Part="1"
-F 0 "U1804" H 7800 2200 50  0000 L CNN
+F 0 "U1102" H 7800 2200 50  0000 L CNN
 F 1 "MC33202" H 7800 2100 50  0000 L CNN
 F 2 "Housings_SOIC:SOIC-8_3.9x4.9mm_Pitch1.27mm" H 7800 1900 50  0001 C CNN
@@
 AR Path="/5DE4AD88/5EE3A0D9/5E6B457F" Ref="U1702"  Part="2"
 AR Path="/5DE4AD88/5EE3A870/5E6B457F" Ref="U1804"  Part="2"
-F 0 "U1804" H 9100 2250 50  0000 L CNN
+F 0 "U1102" H 9100 2250 50  0000 L CNN
 F 1 "MC33202" H 9100 2150 50  0000 L CNN
 F 2 "Housings_SOIC:SOIC-8_3.9x4.9mm_Pitch1.27mm" H 9100 2000 50  0001 C CNN
@@
 AR Path="/5DE4AD88/5EE3A0D9/5E6B7ABF" Ref="C1709"  Part="1"
 AR Path="/5DE4AD88/5EE3A870/5E6B7ABF" Ref="C1812"  Part="1"
-F 0 "C1812" V 7698 1500 50  0000 C CNN
+F 0 "C1108" V 7698 1500 50  0000 C CNN
 F 1 "100n" V 7789 1500 50  0000 C CNN
 F 2 "Capacitors_SMD:C_0603" H 7988 1350 50  0001 C CNN
@@
 AR Path="/5DE4AD88/5EE3A0D9/5E6C400C" Ref="R1712"  Part="1"
 AR Path="/5DE4AD88/5EE3A870/5E6C400C" Ref="R1828"  Part="1"
-F 0 "R1828" V 8350 1850 50  0000 C CNN
+F 0 "R1110" V 8350 1850 50  0000 C CNN
 F 1 "10k" V 8550 1900 50  0000 C CNN
 F 2 "Resistors_SMD:R_0603" V 8380 1900 50  0001 C CNN
@@
 AR Path="/5DE4AD88/5EE3A0D9/5E6C4765" Ref="R1710"  Part="1"
 AR Path="/5DE4AD88/5EE3A870/5E6C4765" Ref="R1826"  Part="1"
-F 0 "R1826" V 7150 1750 50  0000 C CNN
+F 0 "R1108" V 7150 1750 50  0000 C CNN
 F 1 "10k" V 7350 1800 50  0000 C CNN
 F 2 "Resistors_SMD:R_0603" V 7180 1800 50  0001 C CNN
@@
 AR Path="/5DE4AD88/5EE3A0D9/5E6C4D76" Ref="R1714"  Part="1"
 AR Path="/5DE4AD88/5EE3A870/5E6C4D76" Ref="R1830"  Part="1"
-F 0 "R1830" V 8600 1600 50  0000 C CNN
+F 0 "R1112" V 8600 1600 50  0000 C CNN
 F 1 "10k" V 8800 1650 50  0000 C CNN
 F 2 "Resistors_SMD:R_0603" V 8630 1650 50  0001 C CNN
@@
 AR Path="/5DE4AD88/5EE3A0D9/5E6C867B" Ref="R1715"  Part="1"
 AR Path="/5DE4AD88/5EE3A870/5E6C867B" Ref="R1831"  Part="1"
-F 0 "R1831" V 8950 2950 50  0000 C CNN
+F 0 "R1113" V 8950 2950 50  0000 C CNN
 F 1 "10k" V 9150 3000 50  0000 C CNN
 F 2 "Resistors_SMD:R_0603" V 8980 3000 50  0001 C CNN
@@
 AR Path="/5DE4AD88/5EE3A0D9/5E6C8F44" Ref="R1713"  Part="1"
 AR Path="/5DE4AD88/5EE3A870/5E6C8F44" Ref="R1829"  Part="1"
-F 0 "R1829" V 8350 2950 50  0000 C CNN
+F 0 "R1111" V 8350 2950 50  0000 C CNN
 F 1 "10k" V 8550 3000 50  0000 C CNN
 F 2 "Resistors_SMD:R_0603" V 8380 3000 50  0001 C CNN
@@
 AR Path="/5DE4AD88/5EE3A0D9/5E6D075E" Ref="R1716"  Part="1"
 AR Path="/5DE4AD88/5EE3A870/5E6D075E" Ref="R1832"  Part="1"
-F 0 "R1832" V 9650 1950 50  0000 C CNN
+F 0 "R1114" V 9650 1950 50  0000 C CNN
 F 1 "10k" V 9850 2000 50  0000 C CNN
 F 2 "Resistors_SMD:R_0603" V 9680 2000 50  0001 C CNN
@@
 AR Path="/5DE4AD88/5EE3A0D9/5E6D2D7F" Ref="C1710"  Part="1"
 AR Path="/5DE4AD88/5EE3A870/5E6D2D7F" Ref="C1813"  Part="1"
-F 0 "C1813" H 10115 2346 50  0000 L CNN
+F 0 "C1109" H 10115 2346 50  0000 L CNN
 F 1 "100n" H 10115 2255 50  0000 L CNN
 F 2 "Capacitors_SMD:C_0603" H 10038 2150 50  0001 C CNN
@@
 AR Path="/5DE4AD88/5EE3A0D9/5E6D669B" Ref="D1703"  Part="1"
 AR Path="/5DE4AD88/5EE3A870/5E6D669B" Ref="D1802"  Part="1"
-F 0 "D1802" V 8154 3429 50  0000 L CNN
+F 0 "D1102" V 8154 3429 50  0000 L CNN
 F 1 "BZX84Cxx" V 8245 3429 50  0000 L CNN
 F 2 "Diodes_SMD:D_SOT-23_ANK" H 8200 3175 50  0001 C CNN
@@
 AR Path="/5DE4AD88/5EE3A0D9/5E6E4C5D" Ref="C1708"  Part="1"
 AR Path="/5DE4AD88/5EE3A870/5E6E4C5D" Ref="C1811"  Part="1"
-F 0 "C1811" H 7700 3350 50  0000 L CNN
+F 0 "C1107" H 7700 3350 50  0000 L CNN
 F 1 "100n" H 7600 3200 50  0000 L CNN
 F 2 "Capacitors_SMD:C_0603" H 7938 3150 50  0001 C CNN
@@
 AR Path="/5DE4AD88/5EE3A0D9/5E6FB61A" Ref="U1701"  Part="2"
 AR Path="/5DE4AD88/5EE3A870/5E6FB61A" Ref="U1803"  Part="2"
-F 0 "U1803" H 5900 4200 50  0000 L CNN
+F 0 "U1101" H 5900 4200 50  0000 L CNN
 F 1 "LM1458" H 5900 4100 50  0000 L CNN
 F 2 "Housings_SOIC:SOIC-8_3.9x4.9mm_Pitch1.27mm" H 5800 4000 50  0001 C CNN
@@
 AR Path="/5DE4AD88/5EE3A0D9/5E7ABB84" Ref="C1704"  Part="1"
 AR Path="/5DE4AD88/5EE3A870/5E7ABB84" Ref="C1807"  Part="1"
-F 0 "C1807" V 4950 4250 50  0000 C CNN
+F 0 "C1103" V 4950 4250 50  0000 C CNN
 F 1 "100n" V 5250 4250 50  0000 C CNN
 F 2 "Capacitors_SMD:C_0603" H 5138 4100 50  0001 C CNN
@@
 AR Path="/5DE4AD88/5EE3A0D9/5E7AB3BF" Ref="R1705"  Part="1"
 AR Path="/5DE4AD88/5EE3A870/5E7AB3BF" Ref="R1821"  Part="1"
-F 0 "R1821" V 4750 3950 50  0000 C CNN
+F 0 "R1103" V 4750 3950 50  0000 C CNN
 F 1 "10k" V 4950 3900 50  0000 C CNN
 F 2 "Resistors_SMD:R_0603" V 4780 3900 50  0001 C CNN
@@
 AR Path="/5DE4AD88/5EE3A0D9/5E825C1F" Ref="C1702"  Part="1"
 AR Path="/5DE4AD88/5EE3A870/5E825C1F" Ref="C1805"  Part="1"
-F 0 "C1805" V 2900 1500 50  0000 C CNN
+F 0 "C1101" V 2900 1500 50  0000 C CNN
 F 1 "1u" V 3200 1500 50  0000 C CNN
 F 2 "Capacitors_SMD:C_0805" H 3088 1350 50  0001 C CNN
@@
 AR Path="/5DE4AD88/5EE3A0D9/5EDFFDFD" Ref="C2501"  Part="1"
 AR Path="/5DE4AD88/5EE3A870/5EDFFDFD" Ref="C2601"  Part="1"
-F 0 "C2601" H 9165 3296 50  0000 L CNN
+F 0 "C1901" H 9165 3296 50  0000 L CNN
 F 1 "100p" H 9165 3205 50  0000 L CNN
 F 2 "Capacitors_SMD:C_0603" H 9088 3100 50  0001 C CNN
@@
 AR Path="/5DE4AD88/5EE3A0D9/5F717D12" Ref="R1801"  Part="1"
 AR Path="/5DE4AD88/5EE3A870/5F717D12" Ref="R1901"  Part="1"
-F 0 "R1901" V 7550 2950 50  0000 C CNN
+F 0 "R1318" V 7550 2950 50  0000 C CNN
 F 1 "10k" V 7750 3000 50  0000 C CNN
 F 2 "Resistors_SMD:R_0603" V 7580 3000 50  0001 C CNN
