File: cad/fuzz_factory_mod/connectors.sch (KiCad schematic (older format))
At the start: 21 parts, among them J1701 Barrel_Jack_Switch, J1702 Conn_Battery, J1703 CONN_AUDIO_IN, J1704 CONN_AUDIO_OUT, J2801 CONN_AUDIO_OUT_REF, J2802 CONN_EXP_1, J2803 CONN_EXP_2, K2101 Fujitsu-Takamisawa-A_AL, Q1701 DTC114Y, Q1702 DTA114E

Commit message: Continued layout.
Connections:
- net at J1703.5 (R): now also J1702.1 (Pin_1)
- net GNDS: no longer names the net of J1704.5 (R)
- net GNDS: no longer J1702.1 (Pin_1)
Changed lines of the file:
@@
 $EndDescr
-$Comp
-L flax_lib:CLIFF_FCR50051 J1703
-U 1 1 5DE5BD43
-P 2400 1350
-F 0 "J1703" H 2383 1875 50  0000 C CNN
-F 1 "CONN_AUDIO_IN" H 2383 1784 50  0000 C CNN
-F 2 "flax_lib:CLIFF_FCR5005x" H 2500 1200 50  0001 C CNN
-F 3 "" H 2500 1200 50  0001 C CNN
-	1    2400 1350
-	1    0    0    -1
-$EndComp
-$Comp
-L flax_lib:CLIFF_FCR50051 J1704
-U 1 1 5DE5C90E
-P 2400 3350
-F 0 "J1704" H 2450 3900 50  0000 R CNN
-F 1 "CONN_AUDIO_OUT" H 2650 3800 50  0000 R CNN
-F 2 "flax_lib:CLIFF_FCR5005x" H 2500 3200 50  0001 C CNN
-F 3 "" H 2500 3200 50  0001 C CNN
-	1    2400 3350
-	1    0    0    -1
-$EndComp
 $Comp
 L Transistor_BJT:DTC114Y Q1701
@@
 	-1   0    0    -1
 $EndComp
-Wire Wire Line
-	3000 3550 2800 3550
 NoConn ~ 2800 3450
 NoConn ~ 2800 3250
@@
 	2500 4550 2950 4550
 Wire Wire Line
-	3000 4000 3000 3550
-Wire Wire Line
-	2500 4000 3000 4000
-Wire Wire Line
 	2500 4650 2700 4650
 Wire Wire Line
@@
 Connection ~ 2900 1150
 NoConn ~ 2800 1450
-NoConn ~ 2800 1550
 Text Label 8500 3950 2    50   ~ 0
 AUDIO_IN_CONN
@@
 Wire Wire Line
 	4800 5000 4600 5000
-$Comp
-L power:GNDS #PWR01704
-U 1 1 5E6D5175
-P 3100 3550
-F 0 "#PWR01704" H 3100 3300 50  0001 C CNN
-F 1 "GNDS" V 3105 3422 50  0000 R CNN
-F 2 "" H 3100 3550 50  0001 C CNN
-F 3 "" H 3100 3550 50  0001 C CNN
-	1    3100 3550
-	0    -1   -1   0
-$EndComp
-Wire Wire Line
-	3100 3550 3000 3550
-Connection ~ 3000 3550
 $Comp
 L power:GNDPWR #PWR01705
@@
 Wire Wire Line
 	5200 5350 5200 5750
+$Comp
+L flax_lib:CLIFF_FCR50051 J1703
+U 1 1 5DE5BD43
+P 2400 1350
+F 0 "J1703" H 2383 1875 50  0000 C CNN
+F 1 "CONN_AUDIO_IN" H 2383 1784 50  0000 C CNN
+F 2 "flax_lib:CLIFF_FCR5005x" H 2500 1200 50  0001 C CNN
+F 3 "" H 2500 1200 50  0001 C CNN
+	1    2400 1350
+	1    0    0    -1
+$EndComp
+Wire Wire Line
+	2800 1550 4800 1550
+Wire Wire Line
+	4800 1550 4800 4000
+Wire Wire Line
+	2500 4000 4800 4000
+$Comp
+L flax_lib:CLIFF_FCR50051 J1704
+U 1 1 5DE5C90E
+P 2400 3350
+F 0 "J1704" H 2450 3900 50  0000 R CNN
+F 1 "CONN_AUDIO_OUT" H 2650 3800 50  0000 R CNN
+F 2 "flax_lib:CLIFF_FCR5005x" H 2500 3200 50  0001 C CNN
+F 3 "" H 2500 3200 50  0001 C CNN
+	1    2400 3350
+	1    0    0    -1
+$EndComp
+NoConn ~ 2800 3550
 $EndSCHEMATC
