File: cad/fuzz_factory_mod/fuzz_factory_mod_analog/fuzz_factory_ref.sch (KiCad schematic (older format))
At the start: 26 parts

Commit message: Changes architecture.
Corrections on schematic.
Continued Layout placement.
Parts:
- removed Q?: 2N3904, Package_TO_SOT_THT:TO-92_Inline, symbol Transistor_BJT:2N3904
- added Q202: DMMT3904W, TO_SOT_Packages_SMD:SOT-363_SC-70-6, symbol Transistor_BJT:BC846BDW1
- C1601, C1603, C1604: renamed from C?; footprint (none) -> Capacitors_SMD:C_0603
- C1602, C1605, C1606: renamed from C?; footprint (none) -> Capacitors_SMD:CP_Elec_6.3x4.5
- Q1601: renamed from Q?; footprint (none) -> TO_SOT_Packages_SMD:SOT-23
- Q903, Q904: renamed from Q?; value BC857BDW1 -> DMMT3906W; footprint Package_TO_SOT_SMD:SOT-363_SC-70-6 -> TO_SOT_Packages_SMD:SOT-363_SC-70-6
- R1601, R1602, R1603, R1604, R1605, R1606, R1607, R1608, R1609, R1610, R1611, R1612, R1613, R1614, R1615, R1616: renamed from R?; footprint (none) -> Resistors_SMD:R_0603
Connections:
- net labels added: ADC_REF_pol1, ADC_REF_pol2, POL_MEAS_1, POL_MEAS_2
- wire segments 101 -> 105
