File: cad/fuzz_factory_mod/fuzz_factory_mod_interface/interface.sch (KiCad schematic (older format))
At the start: 21 parts, among them U501 TLC6C598-Q1, U502 TLC6C598-Q1

Commit message: Changes architecture.
Corrections on schematic.
Continued Layout placement.
Parts:
- renumbered AFF501 to AFF201, C502 to C201, C503 to C202, R510 to R201, R511 to R202, R512 to R203, R513 to R204, R514 to R205, R515 to R206, R516 to R207, R517 to R208, R518 to R209, R519 to R210, R520 to R211, R521 to R212, R522 to R213, R523 to R214, R524 to R215, R525 to R216, U501 to U201, U502 to U202
Connections:
- net labels removed: +3V3
