File: cad/fuzz_factory_mod/fuzz_factory_mod_interface/fuzz_factory_mod_interface.kicad_pcb (KiCad board)
At the start: 2 copper layers, 68 parts, among them J101 Conn_01x12_Male, J102 Conn_01x12_Male, Q301 DTA123Y, Q302 DTA123Y, Q401 DTA123Y, Q402 DTA123Y, Q501 DTA123Y, Q502 DTA123Y, SW301 PEL12D-4225S-S2024, SW401 PEL12D-4225S-S2024, SW501 PEL12D-4225S-S2024, U201 TLC6C598-Q1, U202 TLC6C598-Q1

Commit message: Continued layout.
Parts:
- J101, J102: moved to B.Cu
- moved R402 139.6 mm to (57.5, 72.1), turned to 180 degrees
- moved R404 139.1 mm to (57.2, 74.6), turned to 180 degrees
- moved R401 133.5 mm to (61.4, 69.7), turned to 180 degrees
- moved R407 132.7 mm to (61.1, 72.2), turned to 180 degrees
- moved C403 131.8 mm to (60.9, 74.6), turned to 180 degrees
- moved SW401 129.0 mm to (50.5, 64.4), turned to 180 degrees
- moved R405 128.4 mm to (65.5, 65.5), turned to 180 degrees
- moved R406 126.6 mm to (64.9, 69.9), turned to 180 degrees
- moved C404 125.5 mm to (64.8, 72.3), turned to 180 degrees
- moved R403 125.4 mm to (69.4, 60.6), turned to 180 degrees
- moved C401 124.3 mm to (64.8, 74.6), turned to 180 degrees
- moved R408 123.2 mm to (69.4, 63.1), turned to 180 degrees
- moved C402 121.5 mm to (69.2, 65.5), turned to 180 degrees
- moved Q401 119.6 mm to (68.9, 69.0), turned to 180 degrees
- moved Q402 116.8 mm to (68.9, 73.5), turned to 180 degrees
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